File: KiCad/duart-rtc.sch (KiCad schematic (older format))
At the start: 4 parts, among them J2 USB_B, U10 DS1501Y, U11 CP2102, U9 68681

Commit message: kprintf working, IDEATA interface started
Parts:
- J2: symbol USB_B -> USB_B-RESCUE-Raven68k
Changed lines of the file:
@@
 EESchema Schematic File Version 2
+LIBS:Raven68k-rescue
 LIBS:Memory_RAM
 LIBS:power
@@
 NoConn ~ 6950 2650
 $Comp
-L USB_B J2
+L USB_B-RESCUE-Raven68k J2
 U 1 1 5A654AF7
 P 9400 1950
