File: prototypes/v1/file5BD91A8D.sch (KiCad schematic (older format))
At the start: 0 parts

Commit message: v1 schematic upates
Parts:
- added JP1, JP2, JP3: Jumper_3_Bridged12, symbol Jumper:Jumper_3_Bridged12
- added U10: 74LS30, symbol 74xx:74LS30
- added U11, U12: KM684000BLP-7L, Package_DIP:DIP-32_W15.24mm, symbol raven:KM684000BLP-7L
- added U13: 74LS138, symbol 74xx:74LS138
- added U14, U15: 28C256, symbol Memory_EEPROM:28C256
- added U3, U? (x2): 74LS04, symbol 74xx:74LS04
- added U4: 74LS20, symbol 74xx:74LS20
- added U6, U? (x3): 74LS00, symbol 74xx:74LS00
Connections:
- new net: U3.2, U6.1
- new net: U13.5 (E2), U6.3
- new net: U3.5, U4.6
- new net: U?.4, U?.8
- new net: U?.10, U?.5
- new net +5V: U10.12, U11.32 (VCC), U12.32 (VCC), U13.16 (VCC), U13.6 (E3), U14.28 (VCC), U15.28 (VCC)
- new net A1: U11.12 (A0), U12.12 (A0), U14.10 (A0), U15.10 (A0)
- new net A10: U11.26 (A9), U12.26 (A9), U14.24 (A9), U15.24 (A9)
- new net A11: U11.23 (A10), U12.23 (A10), U14.21 (A10), U15.21 (A10)
- new net A12: U11.25 (A11), U12.25 (A11), U14.23 (A11), U15.23 (A11)
- new net A13: U11.4 (A12), U12.4 (A12), U14.2 (A12), U15.2 (A12)
- new net A14: U11.28 (A13), U12.28 (A13), U14.26 (A13), U15.26 (A13)
- new net A15: U11.3 (A14), U12.3 (A14), U14.1 (A14), U15.1 (A14)
- new net A16: U11.31 (A15), U12.31 (A15), U6.2
- new net A17: U10.1, U11.2 (A16), U12.2 (A16)
- new net A18: U10.2, U11.30 (A17), U12.30 (A17)
- new net A19: U10.3, U11.1 (A18), U12.1 (A18)
- new net A2: U11.11 (A1), U12.11 (A1), U14.9 (A1), U15.9 (A1)
- new net A20: U10.4, U4.1
- new net A21: U10.5, U4.2
- new net A22: U10.6, U4.4
- new net A23: U10.11, U4.5
- new net A3: U11.10 (A2), U12.10 (A2), U14.8 (A2), U15.8 (A2)
- new net A4: U11.9 (A3), U12.9 (A3), U14.7 (A3), U15.7 (A3)
- new net A5: U11.8 (A4), U12.8 (A4), U14.6 (A4), U15.6 (A4)
- new net A6: U11.7 (A5), U12.7 (A5), U14.5 (A5), U15.5 (A5)
- new net A7: U11.6 (A6), U12.6 (A6), U13.1 (A0), U14.4 (A6), U15.4 (A6)
- new net A8: U11.5 (A7), U12.5 (A7), U13.2 (A1), U14.3 (A7), U15.3 (A7)
- new net A9: U11.27 (A8), U12.27 (A8), U13.3 (A2), U14.25 (A8), U15.25 (A8)
- new net D0: U11.13 (D0), U14.11 (D0)
- new net D1: U11.14 (D1), U14.12 (D1)
- new net D10: U12.15 (D2), U15.13 (D2)
- new net D11: U12.17 (D3), U15.15 (D3)
- new net D12: U12.18 (D4), U15.16 (D4)
- new net D13: U12.19 (D5), U15.17 (D5)
- new net D14: U12.20 (D6), U15.18 (D6)
- new net D15: U12.21 (D7), U15.19 (D7)
- new net D2: U11.15 (D2), U14.13 (D2)
- new net D3: U11.17 (D3), U14.15 (D3)
- new net D4: U11.18 (D4), U14.16 (D4)
- new net D5: U11.19 (D5), U14.17 (D5)
- new net D6: U11.20 (D6), U14.18 (D6)
- new net D7: U11.21 (D7), U14.19 (D7)
- new net D8: U12.13 (D0), U15.11 (D0)
- new net D9: U12.14 (D1), U15.12 (D1)
- new net DUART_CS: JP2.2 (C)
- new net DUART_CS_JMPR: JP2.1 (A), U13.15 (O0)
- new net EXT_DUART_CS: JP2.3 (B)
- new net EXT_RAM_CS: JP3.3 (B)
- new net EXT_ROM_CS: JP1.3 (B)
- new net GND: U11.16 (GND), U12.16 (GND), U13.4 (E1), U13.8 (GND), U14.14 (GND), U15.14 (GND)
- new net OE: U11.24 (~OE), U12.24 (~OE), U14.22 (~OE), U15.22 (~OE)
- new net RAM_CS: JP3.2 (C), U?.9
- new net RAM_CS_JMPR: JP3.1 (A), U3.6
- new net RAM_UDS: U?.6
- new net ROM_CS: JP1.2 (C), U14.20 (~CS), U15.20 (~CS), U3.1
- new net ROM_CS_JMPR: JP1.1 (A), U10.8
- new net RW: U11.29 (~WE), U12.29 (~WE), U14.27 (~WE), U15.27 (~WE)
- new net UDS: U?.11
- no-connect marks 0 -> 7
