File: prototypes/v1/raven-prototypes.kicad_pcb (KiCad board)
At the start: 2 copper layers, 163 x 112 mm, 46 parts, among them J1 Serial_Connections, J2 Ext_Signal, J3 770997-1, U1 68010D, U10 MCP100-485D, U11 74LS20, U12 74LS30, U13 74LS138, U14 74LS04, U15 74LS00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

Commit message: gerbers created, Rev 0 sent to manufacturer
Routing:
- net GND: track 776.1 -> 906.7 mm, vias 0 -> 5
Changed lines of the file:
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@@
     (thickness 1.6)
     (drawings 7)
-    (tracks 2327)
+    (tracks 2353)
     (zones 0)
     (modules 46)
@@
   (segment (start 116.04 45.3669) (end 121.77274 39.63416) (width 0.1) (layer B.Cu) (net 1))
   (segment (start 121.77274 39.63416) (end 126.69774 39.63416) (width 0.1) (layer B.Cu) (net 1))
-  (segment (start 126.69774 39.63416) (end 143.54048 39.63416) (width 0.1) (layer F.Cu) (net 1))
   (via (at 155.09748 45.21454) (size 0.8) (drill 0.4) (layers F.Cu B.Cu) (net 1))
-  (segment (start 143.54048 39.63416) (end 149.12086 45.21454) (width 0.1) (layer F.Cu) (net 1))
-  (segment (start 149.12086 45.21454) (end 155.09748 45.21454) (width 0.1) (layer F.Cu) (net 1))
   (segment (start 151.558 48.75402) (end 151.558 49.4346) (width 0.1) (layer B.Cu) (net 1))
   (segment (start 155.09748 45.21454) (end 151.558 48.75402) (width 0.1) (layer B.Cu) (net 1))
+  (segment (start 149.065638 45.21454) (end 154.531795 45.21454) (width 0.1) (layer F.Cu) (net 1))
+  (segment (start 154.531795 45.21454) (end 155.09748 45.21454) (width 0.1) (layer F.Cu) (net 1))
+  (segment (start 143.485258 39.63416) (end 149.065638 45.21454) (width 0.1) (layer F.Cu) (net 1))
+  (segment (start 126.69774 39.63416) (end 143.485258 39.63416) (width 0.1) (layer F.Cu) (net 1))
   (segment (start 86.26 74.5) (end 87.3681 73.3919) (width 0.1) (layer B.Cu) (net 2))
   (segment (start 87.3681 54.6081) (end 86.26 53.5) (width 0.1) (layer B.Cu) (net 2))
@@
   (segment (start 143.524001 89.231401) (end 144.324 90.0314) (width 0.1) (layer F.Cu) (net 2))
   (segment (start 87.3681 73.3919) (end 87.3681 54.6081) (width 0.1) (layer B.Cu) (net 2))
+  (via (at 210.4517 65.9384) (size 0.8) (drill 0.4) (layers F.Cu B.Cu) (net 2))
+  (segment (start 216 87.24) (end 210.4517 81.6917) (width 0.1) (layer F.Cu) (net 2))
+  (segment (start 210.4517 81.6917) (end 210.4517 65.9384) (width 0.1) (layer F.Cu) (net 2))
+  (via (at 198.84136 42.29354) (size 0.8) (drill 0.4) (layers F.Cu B.Cu) (net 2))
+  (segment (start 210.4517 65.9384) (end 210.4517 53.90388) (width 0.1) (layer B.Cu) (net 2))
+  (segment (start 210.4517 53.90388) (end 198.84136 42.29354) (width 0.1) (layer B.Cu) (net 2))
+  (via (at 175.6029 42.6593) (size 0.8) (drill 0.4) (layers F.Cu B.Cu) (net 2))
+  (segment (start 198.84136 42.29354) (end 175.96866 42.29354) (width 0.1) (layer F.Cu) (net 2))
+  (segment (start 175.96866 42.29354) (end 175.6029 42.6593) (width 0.1) (layer F.Cu) (net 2))
+  (segment (start 175.037215 42.6593) (end 174.905135 42.79138) (width 0.1) (layer B.Cu) (net 2))
+  (segment (start 175.6029 42.6593) (end 175.037215 42.6593) (width 0.1) (layer B.Cu) (net 2))
+  (segment (start 174.905135 42.79138) (end 153.84018 42.79138) (width 0.1) (layer B.Cu) (net 2))
+  (via (at 149.06498 44.25188) (size 0.8) (drill 0.4) (layers F.Cu B.Cu) (net 2))
+  (segment (start 153.84018 42.79138) (end 152.37968 44.25188) (width 0.1) (layer B.Cu) (net 2))
+  (segment (start 152.37968 44.25188) (end 149.06498 44.25188) (width 0.1) (layer B.Cu) (net 2))
+  (segment (start 148.664981 43.851881) (end 148.664981 43.653761) (width 0.1) (layer F.Cu) (net 2))
+  (segment (start 149.06498 44.25188) (end 148.664981 43.851881) (width 0.1) (layer F.Cu) (net 2))
+  (segment (start 148.664981 43.653761) (end 143.86306 38.85184) (width 0.1) (layer F.Cu) (net 2))
+  (segment (start 143.86306 38.85184) (end 133.11632 38.85184) (width 0.1) (layer F.Cu) (net 2))
+  (via (at 133.11632 38.85184) (size 0.8) (drill 0.4) (layers F.Cu B.Cu) (net 2))
+  (segment (start 126.60126 45.3669) (end 126.2 45.3669) (width 0.1) (layer B.Cu) (net 2))
+  (segment (start 133.11632 38.85184) (end 126.60126 45.3669) (width 0.1) (layer B.Cu) (net 2))
   (segment (start 172.0767 38.2295) (end 172.0767 38.0015) (width 0.1) (layer B.Cu) (net 3))
   (segment (start 172.0767 38.0015) (end 170.5845 36.5093) (width 0.1) (layer B.Cu) (net 3))
@@
   (segment (start 157.937 38.2295) (end 156.8367 38.2295) (width 0.1) (layer F.Cu) (net 9))
   (segment (start 69 123.62) (end 69 122.5697) (width 0.1) (layer F.Cu) (net 9))
-  (segment (start 155.397 38.2295) (end 154.2967 38.2295) (width 0.1) (layer B.Cu) (net 10))
-  (segment (start 69 126.16) (end 70.0503 126.16) (width 0.1) (layer B.Cu) (net 10))
-  (segment (start 70.0503 126.16) (end 76.1906 120.0197) (width 0.1) (layer B.Cu) (net 10))
-  (segment (start 76.1906 120.0197) (end 77.8801 120.0197) (width 0.1) (layer B.Cu) (net 10))
-  (segment (start 77.8801 120.0197) (end 78.1827 120.3223) (width 0.1) (layer B.Cu) (net 10))
-  (segment (start 78.1827 120.3223) (end 92.8651 120.3223) (width 0.1) (layer B.Cu) (net 10))
-  (segment (start 92.8651 120.3223) (end 99.3574 113.83) (width 0.1) (layer B.Cu) (net 10))
-  (segment (start 99.3574 113.83) (end 99.3574 111.6496) (width 0.1) (layer B.Cu) (net 10))
+  (segment (start 69 126.16) (end 75.1403 120.0197) (width 0.1) (layer B.Cu) (net 10))
+  (segment (start 102.9405 66.6546) (end 131.3656 38.2295) (width 0.1) (layer B.Cu) (net 10))
+  (segment (start 131.3656 38.2295) (end 132.776658 38.2295) (width 0.1) (layer B.Cu) (net 10))
+  (segment (start 132.776658 38.2295) (end 132.804319 38.201839) (width 0.1) (layer B.Cu) (net 10))
+  (segment (start 132.804319 38.201839) (end 133.428321 38.201839) (width 0.1) (layer B.Cu) (net 10))
+  (segment (start 154.447 38.2295) (end 155.397 38.2295) (width 0.1) (layer B.Cu) (net 10))
+  (segment (start 133.428321 38.201839) (end 133.455982 38.2295) (width 0.1) (layer B.Cu) (net 10))
+  (segment (start 102.9405 108.5666) (end 102.9405 66.6546) (width 0.1) (layer B.Cu) (net 10))
   (segment (start 99.3574 111.6496) (end 100.957 110.05) (width 0.1) (layer B.Cu) (net 10))
-  (segment (start 100.957 110.05) (end 101.4571 110.05) (width 0.1) (layer B.Cu) (net 10))
+  (segment (start 92.8651 120.3223) (end 99.3574 113.83) (width 0.1) (layer B.Cu) (net 10))
+  (segment (start 133.455982 38.2295) (end 154.447 38.2295) (width 0.1) (layer B.Cu) (net 10))
   (segment (start 101.4571 110.05) (end 102.9405 108.5666) (width 0.1) (layer B.Cu) (net 10))
-  (segment (start 102.9405 108.5666) (end 102.9405 66.6546) (width 0.1) (layer B.Cu) (net 10))
-  (segment (start 102.9405 66.6546) (end 131.3656 38.2295) (width 0.1) (layer B.Cu) (net 10))
-  (segment (start 131.3656 38.2295) (end 154.2967 38.2295) (width 0.1) (layer B.Cu) (net 10))
+  (segment (start 100.957 110.05) (end 101.4571 110.05) (width 0.1) (layer B.Cu) (net 10))
+  (segment (start 99.3574 113.83) (end 99.3574 111.6496) (width 0.1) (layer B.Cu) (net 10))
+  (segment (start 78.1827 120.3223) (end 92.8651 120.3223) (width 0.1) (layer B.Cu) (net 10))
+  (segment (start 77.8801 120.0197) (end 78.1827 120.3223) (width 0.1) (layer B.Cu) (net 10))
+  (segment (start 75.1403 120.0197) (end 77.8801 120.0197) (width 0.1) (layer B.Cu) (net 10))
   (segment (start 69.8295 48.0903) (end 69.8295 47.9815) (width 0.1) (layer F.Cu) (net 11))
   (segment (start 69.8295 47.9815) (end 71.502 46.309) (width 0.1) (layer F.Cu) (net 11))
