File: prototypes/v1/raven-prototypes.sch (KiCad schematic (older format))
At the start: 9 parts

Commit message: v1 schematic upates
Parts:
- removed U?: 74LS10, symbol 74xx:74LS10
- removed U?: 68681, symbol Interface:68681
- added U3: 74LS04, symbol 74xx:74LS04
- gave numbers to parts that had none: 7
Connections:
- net RW: now also U3.3
- net FC2: now reaches U9.26 (FC2)
- net FC2: now also U1.1
- net FC1: now reaches U9.27 (FC1)
- net FC1: now also U1.2
- net FC0: now reaches U9.28 (FC0)
- net FC0: now also U1.13
- new net OE: U3.4
- no-connect marks 22 -> 21
Other:
- moved on the sheet: U1A, U2, U5, X1, X2

Commit message: finish logic
Parts:
- renumbered U2 to U1, U3 to U2, U5 to U3, U1 to U4, U8 to U5, U9 to U6
Changed lines of the file:
@@
 $EndDescr
 $Comp
-L CPU_NXP_68000:68010D U9
+L CPU_NXP_68000:68010D U6
 U 1 1 5BBD648E
 P 11300 3650
-F 0 "U9" H 11700 6100 50  0000 C CNN
+F 0 "U6" H 11700 6100 50  0000 C CNN
 F 1 "68010D" H 11700 6000 50  0000 C CNN
 F 2 "" H 11300 3650 50  0001 C CNN
@@
 Connection ~ 11300 1200
 $Comp
-L power:GND #PWR0101
+L power:GND #PWR08
 U 1 1 5BBDC0F1
 P 11550 6200
-F 0 "#PWR0101" H 11550 5950 50  0001 C CNN
+F 0 "#PWR08" H 11550 5950 50  0001 C CNN
 F 1 "GND" H 11555 6027 50  0000 C CNN
 F 2 "" H 11550 6200 50  0001 C CNN
@@
 	3150 6300 3400 6300
 $Comp
-L power:GND #PWR0102
+L power:GND #PWR05
 U 1 1 5BBF29FB
 P 3550 7700
-F 0 "#PWR0102" H 3550 7450 50  0001 C CNN
+F 0 "#PWR05" H 3550 7450 50  0001 C CNN
 F 1 "GND" H 3555 7527 50  0000 C CNN
 F 2 "" H 3550 7700 50  0001 C CNN
@@
 $EndComp
 $Comp
-L 74xx:74LS148 U2
+L 74xx:74LS148 U1
 U 1 1 5BBF46DF
 P 3400 7000
-F 0 "U2" H 3400 7878 50  0000 C CNN
+F 0 "U1" H 3400 7878 50  0000 C CNN
 F 1 "74LS148" H 3400 7787 50  0000 C CNN
 F 2 "" H 3400 7000 50  0001 C CNN
@@
 NoConn ~ 3900 7200
 $Comp
-L 74xx:74LS10 U1
+L 74xx:74LS10 U4
 U 1 1 5BBFB7E8
 P 6800 7200
-F 0 "U1" H 6800 6883 50  0000 C CNN
+F 0 "U4" H 6800 6883 50  0000 C CNN
 F 1 "74LS10" H 6800 6974 50  0000 C CNN
 F 2 "" H 6800 7200 50  0001 C CNN
@@
 IPL2
 $Comp
-L power:GND #PWR0103
+L power:GND #PWR03
 U 1 1 5BC06A34
 P 2700 6600
-F 0 "#PWR0103" H 2700 6350 50  0001 C CNN
+F 0 "#PWR03" H 2700 6350 50  0001 C CNN
 F 1 "GND" H 2705 6427 50  0000 C CNN
 F 2 "" H 2700 6600 50  0001 C CNN
@@
 	2900 6600 2700 6600
 $Comp
-L power:GND #PWR0104
+L power:GND #PWR04
 U 1 1 5BC08D08
 P 2700 7400
-F 0 "#PWR0104" H 2700 7150 50  0001 C CNN
+F 0 "#PWR04" H 2700 7150 50  0001 C CNN
 F 1 "GND" H 2705 7227 50  0000 C CNN
 F 2 "" H 2700 7400 50  0001 C CNN
@@
 FC
 $Comp
-L 74xx:74LS138 U5
+L 74xx:74LS138 U3
 U 1 1 5BC1A1E7
 P 5700 6900
-F 0 "U5" H 5700 7678 50  0000 C CNN
+F 0 "U3" H 5700 7678 50  0000 C CNN
 F 1 "74LS138" H 5700 7587 50  0000 C CNN
 F 2 "" H 5700 6900 50  0001 C CNN
@@
 	5550 6300 5700 6300
 $Comp
-L power:GND #PWR0106
+L power:GND #PWR06
 U 1 1 5BC706B3
 P 5850 7650
-F 0 "#PWR0106" H 5850 7400 50  0001 C CNN
+F 0 "#PWR06" H 5850 7400 50  0001 C CNN
 F 1 "GND" H 5855 7477 50  0000 C CNN
 F 2 "" H 5850 7650 50  0001 C CNN
@@
 +5V
 $Comp
-L power:GND #PWR0107
+L power:GND #PWR02
 U 1 1 5BC953AC
 P 1300 7550
-F 0 "#PWR0107" H 1300 7300 50  0001 C CNN
+F 0 "#PWR02" H 1300 7300 50  0001 C CNN
 F 1 "GND" H 1305 7377 50  0000 C CNN
 F 2 "" H 1300 7550 50  0001 C CNN
@@
 	10300 4450 10050 4450
 $Comp
-L Power_Supervisor:MCP100-485D U8
+L Power_Supervisor:MCP100-485D U5
 U 1 1 5BCBD7C2
 P 9300 4950
-F 0 "U8" H 9070 4996 50  0000 R CNN
+F 0 "U5" H 9070 4996 50  0000 R CNN
 F 1 "MCP100-485D" H 9070 4905 50  0000 R CNN
 F 2 "" H 8900 5100 50  0001 C CNN
@@
 	9200 4500 9200 4550
 $Comp
-L power:GND #PWR0108
+L power:GND #PWR07
 U 1 1 5BCD185A
 P 9350 5350
-F 0 "#PWR0108" H 9350 5100 50  0001 C CNN
+F 0 "#PWR07" H 9350 5100 50  0001 C CNN
 F 1 "GND" H 9355 5177 50  0000 C CNN
 F 2 "" H 9350 5350 50  0001 C CNN
@@
 +5V
 $Comp
-L power:GND #PWR0109
+L power:GND #PWR01
 U 1 1 5BD0D66E
 P 1250 6400
-F 0 "#PWR0109" H 1250 6150 50  0001 C CNN
+F 0 "#PWR01" H 1250 6150 50  0001 C CNN
 F 1 "GND" H 1255 6227 50  0000 C CNN
 F 2 "" H 1250 6400 50  0001 C CNN
@@
 $EndSheet
 $Comp
-L 74xx:74LS04 U3
+L 74xx:74LS04 U2
 U 2 1 5BC27323
 P 5300 1250
-F 0 "U3" H 5300 1567 50  0000 C CNN
+F 0 "U2" H 5300 1567 50  0000 C CNN
 F 1 "74LS04" H 5300 1476 50  0000 C CNN
 F 2 "" H 5300 1250 50  0001 C CNN
@@
 Wire Wire Line
 	5700 7650 5850 7650
-Wire Bus Line
-	10000 1750 10000 2050
-Wire Bus Line
-	4200 6600 4200 6900
-Wire Bus Line
-	10050 2650 10050 2950
-Wire Bus Line
-	7350 7100 7350 7400
-Wire Bus Line
-	6500 6600 6500 6900
-Wire Bus Line
-	12650 1400 12650 3750
-Wire Bus Line
-	12650 3850 12650 5450
 Text Label 10200 2650 0    50   ~ 0
 FC0
@@
 Text Label 7150 7300 0    50   ~ 0
 FC2
+Wire Bus Line
+	10000 1750 10000 2050
+Wire Bus Line
+	4200 6600 4200 6900
+Wire Bus Line
+	10050 2650 10050 2950
+Wire Bus Line
+	7350 7100 7350 7400
+Wire Bus Line
+	6500 6600 6500 6900
+Wire Bus Line
+	12650 1400 12650 3750
+Wire Bus Line
+	12650 3850 12650 5450
 $EndSCHEMATC

Commit message: optimized logic
Parts:
- added unit 2 of U7
- added unit 3 of U7
- U1: renamed from U6; footprint (none) -> Package_DIP:DIP-64_W22.86mm
- X1, X2: footprint Oscillator:Oscillator_DIP-14 -> (none)
- renumbered U5 to U10, U1 to U2, U2 to U7, U3 to U8, U4 to U9
Connections:
- net DUART_CLK: now also U7.4; no longer X1.8 (OUT)
- net OE: now also U7.2; no longer U7.4
- net RW: now also U7.1; no longer U7.3
- net SYS_CLK: now also U7.6; no longer X2.8 (OUT)
- new net: U7.5, X2.8 (OUT)
- new net: U7.3, X1.8 (OUT)
Other:
- moved on the sheet: X1, X2
Changed lines of the file:
@@
 $EndDescr
 $Comp
-L CPU_NXP_68000:68010D U6
+L CPU_NXP_68000:68010D U1
 U 1 1 5BBD648E
 P 11300 3650
-F 0 "U6" H 11700 6100 50  0000 C CNN
+F 0 "U1" H 11700 6100 50  0000 C CNN
 F 1 "68010D" H 11700 6000 50  0000 C CNN
-F 2 "" H 11300 3650 50  0001 C CNN
+F 2 "Package_DIP:DIP-64_W22.86mm" H 11300 3650 50  0001 C CNN
 F 3 "https://www.nxp.com/docs/en/reference-manual/MC68000UM.pdf" H 11300 3650 50  0001 C CNN
 	1    11300 3650
@@
 L Oscillator:CXO_DIP14 X2
 U 1 1 5BBD8DE1
-P 1200 7200
-F 0 "X2" H 1500 7050 50  0000 L CNN
-F 1 "8 MHZ" H 1450 6950 50  0000 L CNN
-F 2 "Oscillator:Oscillator_DIP-14" H 1650 6850 50  0001 C CNN
-F 3 "http://cdn-reichelt.de/documents/datenblatt/B400/OSZI.pdf" H 1100 7200 50  0001 C CNN
-	1    1200 7200
+P 5850 3900
+F 0 "X2" H 6150 3750 50  0000 L CNN
+F 1 "8 MHZ" H 6100 3650 50  0000 L CNN
+F 2 "" H 6300 3550 50  0001 C CNN
+F 3 "http://cdn-reichelt.de/documents/datenblatt/B400/OSZI.pdf" H 5750 3900 50  0001 C CNN
+	1    5850 3900
 	1    0    0    -1
 $EndComp
@@
 L power:GND #PWR08
 U 1 1 5BBDC0F1
-P 11550 6200
-F 0 "#PWR08" H 11550 5950 50  0001 C CNN
-F 1 "GND" H 11555 6027 50  0000 C CNN
-F 2 "" H 11550 6200 50  0001 C CNN
-F 3 "" H 11550 6200 50  0001 C CNN
-	1    11550 6200
-	1    0    0    -1
-$EndComp
-Wire Wire Line
-	11400 6050 11400 6200
-Wire Wire Line
-	11400 6200 11550 6200
+P 11500 6200
+F 0 "#PWR08" H 11500 5950 50  0001 C CNN
+F 1 "GND" H 11505 6027 50  0000 C CNN
+F 2 "" H 11500 6200 50  0001 C CNN
+F 3 "" H 11500 6200 50  0001 C CNN
+	1    11500 6200
+	1    0    0    -1
+$EndComp
 Wire Wire Line
 	11300 6050 11300 6200
-Wire Wire Line
-	11300 6200 11400 6200
-Connection ~ 11400 6200
-Text GLabel 1700 7200 2    50   Output ~ 0
+Text GLabel 7250 3900 2    50   Output ~ 0
 SYS_CLK
 Wire Wire Line
-	1500 7200 1700 7200
+	6150 3900 6350 3900
 Text GLabel 10150 1450 0    50   Input ~ 0
 SYS_CLK
@@
 	3150 6300 3400 6300
 $Comp
-L power:GND #PWR05
+L power:GND #PWR02
 U 1 1 5BBF29FB
 P 3550 7700
-F 0 "#PWR05" H 3550 7450 50  0001 C CNN
+F 0 "#PWR02" H 3550 7450 50  0001 C CNN
 F 1 "GND" H 3555 7527 50  0000 C CNN
 F 2 "" H 3550 7700 50  0001 C CNN
@@
 $EndComp
 $Comp
-L 74xx:74LS148 U1
+L 74xx:74LS148 U2
 U 1 1 5BBF46DF
 P 3400 7000
-F 0 "U1" H 3400 7878 50  0000 C CNN
+F 0 "U2" H 3400 7878 50  0000 C CNN
 F 1 "74LS148" H 3400 7787 50  0000 C CNN
 F 2 "" H 3400 7000 50  0001 C CNN
@@
 NoConn ~ 3900 7200
 $Comp
-L 74xx:74LS10 U4
+L 74xx:74LS10 U9
 U 1 1 5BBFB7E8
 P 6800 7200
-F 0 "U4" H 6800 6883 50  0000 C CNN
+F 0 "U9" H 6800 6883 50  0000 C CNN
 F 1 "74LS10" H 6800 6974 50  0000 C CNN
 F 2 "" H 6800 7200 50  0001 C CNN
@@
 IPL2
 $Comp
-L power:GND #PWR03
+L power:GND #PWR01
 U 1 1 5BC06A34
 P 2700 6600
-F 0 "#PWR03" H 2700 6350 50  0001 C CNN
+F 0 "#PWR01" H 2700 6350 50  0001 C CNN
 F 1 "GND" H 2705 6427 50  0000 C CNN
 F 2 "" H 2700 6600 50  0001 C CNN
@@
 Wire Wire Line
 	2900 6600 2700 6600
-$Comp
-L power:GND #PWR04
-U 1 1 5BC08D08
-P 2700 7400
-F 0 "#PWR04" H 2700 7150 50  0001 C CNN
-F 1 "GND" H 2705 7227 50  0000 C CNN
-F 2 "" H 2700 7400 50  0001 C CNN
-F 3 "" H 2700 7400 50  0001 C CNN
-	1    2700 7400
-	1    0    0    -1
-$EndComp
-Wire Wire Line
-	2700 7400 2900 7400
 Wire Wire Line
 	10300 2650 10150 2650
@@
 FC
 $Comp
-L 74xx:74LS138 U3
+L 74xx:74LS138 U8
 U 1 1 5BC1A1E7
 P 5700 6900
-F 0 "U3" H 5700 7678 50  0000 C CNN
+F 0 "U8" H 5700 7678 50  0000 C CNN
 F 1 "74LS138" H 5700 7587 50  0000 C CNN
 F 2 "" H 5700 6900 50  0001 C CNN
@@
 	5550 6300 5700 6300
 $Comp
-L power:GND #PWR06
+L power:GND #PWR03
 U 1 1 5BC706B3
 P 5850 7650
-F 0 "#PWR06" H 5850 7400 50  0001 C CNN
+F 0 "#PWR03" H 5850 7400 50  0001 C CNN
 F 1 "GND" H 5855 7477 50  0000 C CNN
 F 2 "" H 5850 7650 50  0001 C CNN
@@
 NoConn ~ 2900 7200
 NoConn ~ 2900 7300
-Text GLabel 1050 6850 0    50   Input ~ 0
-+5V
-$Comp
-L power:GND #PWR02
+Text GLabel 5700 3550 0    50   Input ~ 0
++5V
+$Comp
+L power:GND #PWR05
 U 1 1 5BC953AC
-P 1300 7550
-F 0 "#PWR02" H 1300 7300 50  0001 C CNN
-F 1 "GND" H 1305 7377 50  0000 C CNN
-F 2 "" H 1300 7550 50  0001 C CNN
-F 3 "" H 1300 7550 50  0001 C CNN
-	1    1300 7550
-	1    0    0    -1
-$EndComp
-Wire Wire Line
-	1200 7500 1200 7550
-Wire Wire Line
-	1200 7550 1300 7550
-Wire Wire Line
-	1050 6850 1200 6850
-Wire Wire Line
-	1200 6850 1200 6900
-NoConn ~ 900  7200
+P 5950 4250
+F 0 "#PWR05" H 5950 4000 50  0001 C CNN
+F 1 "GND" H 5955 4077 50  0000 C CNN
+F 2 "" H 5950 4250 50  0001 C CNN
+F 3 "" H 5950 4250 50  0001 C CNN
+	1    5950 4250
+	1    0    0    -1
+$EndComp
+Wire Wire Line
+	5850 4200 5850 4250
+Wire Wire Line
+	5850 4250 5950 4250
+Wire Wire Line
+	5700 3550 5850 3550
+Wire Wire Line
+	5850 3550 5850 3600
+NoConn ~ 5550 3900
 Text GLabel 10050 3350 0    50   Input ~ 0
 +5V
@@
 	10300 4450 10050 4450
 $Comp
-L Power_Supervisor:MCP100-485D U5
+L Power_Supervisor:MCP100-485D U10
 U 1 1 5BCBD7C2
 P 9300 4950
-F 0 "U5" H 9070 4996 50  0000 R CNN
+F 0 "U10" H 9070 4996 50  0000 R CNN
 F 1 "MCP100-485D" H 9070 4905 50  0000 R CNN
 F 2 "" H 8900 5100 50  0001 C CNN
@@
 	9200 4500 9200 4550
 $Comp
-L power:GND #PWR07
+L power:GND #PWR06
 U 1 1 5BCD185A
 P 9350 5350
-F 0 "#PWR07" H 9350 5100 50  0001 C CNN
+F 0 "#PWR06" H 9350 5100 50  0001 C CNN
 F 1 "GND" H 9355 5177 50  0000 C CNN
 F 2 "" H 9350 5350 50  0001 C CNN
@@
 L Oscillator:CXO_DIP14 X1
 U 1 1 5BD0D5E0
-P 1150 6050
-F 0 "X1" H 1450 5900 50  0000 L CNN
-F 1 "3.6864 MHZ" H 1400 5800 50  0000 L CNN
-F 2 "Oscillator:Oscillator_DIP-14" H 1600 5700 50  0001 C CNN
-F 3 "http://cdn-reichelt.de/documents/datenblatt/B400/OSZI.pdf" H 1050 6050 50  0001 C CNN
-	1    1150 6050
-	1    0    0    -1
-$EndComp
-Text GLabel 1000 5700 0    50   Input ~ 0
-+5V
-$Comp
-L power:GND #PWR01
+P 5800 2750
+F 0 "X1" H 6100 2600 50  0000 L CNN
+F 1 "3.6864 MHZ" H 6050 2500 50  0000 L CNN
+F 2 "" H 6250 2400 50  0001 C CNN
+F 3 "http://cdn-reichelt.de/documents/datenblatt/B400/OSZI.pdf" H 5700 2750 50  0001 C CNN
+	1    5800 2750
+	1    0    0    -1
+$EndComp
+Text GLabel 5650 2400 0    50   Input ~ 0
++5V
+$Comp
+L power:GND #PWR04
 U 1 1 5BD0D66E
-P 1250 6400
-F 0 "#PWR01" H 1250 6150 50  0001 C CNN
-F 1 "GND" H 1255 6227 50  0000 C CNN
-F 2 "" H 1250 6400 50  0001 C CNN
-F 3 "" H 1250 6400 50  0001 C CNN
-	1    1250 6400
-	1    0    0    -1
-$EndComp
-Text GLabel 1700 6050 2    50   Output ~ 0
+P 5900 3100
+F 0 "#PWR04" H 5900 2850 50  0001 C CNN
+F 1 "GND" H 5905 2927 50  0000 C CNN
+F 2 "" H 5900 3100 50  0001 C CNN
+F 3 "" H 5900 3100 50  0001 C CNN
+	1    5900 3100
+	1    0    0    -1
+$EndComp
+Text GLabel 7200 2750 2    50   Output ~ 0
 DUART_CLK
 Wire Wire Line
-	1000 5700 1150 5700
-Wire Wire Line
-	1150 5700 1150 5750
-Wire Wire Line
-	1700 6050 1450 6050
-Wire Wire Line
-	1150 6350 1150 6400
-Wire Wire Line
-	1150 6400 1250 6400
-NoConn ~ 850  6050
-NoConn ~ 5650 1100
+	5650 2400 5800 2400
+Wire Wire Line
+	5800 2400 5800 2450
+Wire Wire Line
+	6350 2750 6100 2750
+Wire Wire Line
+	5800 3050 5800 3100
+Wire Wire Line
+	5800 3100 5900 3100
+NoConn ~ 5500 2750
+NoConn ~ 6550 1400
 $Sheet
 S 600  650  900  1200
@@
 $EndSheet
 $Comp
-L 74xx:74LS04 U2
-U 2 1 5BC27323
-P 5300 1250
-F 0 "U2" H 5300 1567 50  0000 C CNN
-F 1 "74LS04" H 5300 1476 50  0000 C CNN
-F 2 "" H 5300 1250 50  0001 C CNN
-F 3 "http://www.ti.com/lit/gpn/sn74LS04" H 5300 1250 50  0001 C CNN
-	2    5300 1250
-	1    0    0    -1
-$EndComp
-Text GLabel 4850 1250 0    50   Input ~ 0
+L 74xx:74LS04 U7
+U 1 1 5BC27323
+P 6200 1550
+F 0 "U7" H 6200 1867 50  0000 C CNN
+F 1 "74LS04" H 6200 1776 50  0000 C CNN
+F 2 "" H 6200 1550 50  0001 C CNN
+F 3 "http://www.ti.com/lit/gpn/sn74LS04" H 6200 1550 50  0001 C CNN
+	1    6200 1550
+	1    0    0    -1
+$EndComp
+Text GLabel 5750 1550 0    50   Input ~ 0
 RW
 Wire Wire Line
-	4850 1250 5000 1250
-Wire Wire Line
-	5600 1250 5750 1250
-Text GLabel 5750 1250 2    50   Output ~ 0
+	5750 1550 5900 1550
+Wire Wire Line
+	6500 1550 6650 1550
+Text GLabel 6650 1550 2    50   Output ~ 0
 OE
 $Sheet
@@
 Text Label 7150 7300 0    50   ~ 0
 FC2
+Wire Wire Line
+	2900 7400 2900 7700
+Wire Wire Line
+	2900 7700 3400 7700
+Connection ~ 3400 7700
+$Comp
+L power:GND #PWR07
+U 1 1 5BD68CBC
+P 11200 6200
+F 0 "#PWR07" H 11200 5950 50  0001 C CNN
+F 1 "GND" H 11205 6027 50  0000 C CNN
+F 2 "" H 11200 6200 50  0001 C CNN
+F 3 "" H 11200 6200 50  0001 C CNN
+	1    11200 6200
+	1    0    0    -1
+$EndComp
+Wire Wire Line
+	11200 6200 11300 6200
+Wire Wire Line
+	11400 6200 11500 6200
+Wire Wire Line
+	11400 6050 11400 6200
+$Comp
+L 74xx:74LS04 U7
+U 2 1 5C0FE576
+P 6650 2750
+F 0 "U7" H 6650 3067 50  0000 C CNN
+F 1 "74LS04" H 6650 2976 50  0000 C CNN
+F 2 "" H 6650 2750 50  0001 C CNN
+F 3 "http://www.ti.com/lit/gpn/sn74LS04" H 6650 2750 50  0001 C CNN
+	2    6650 2750
+	1    0    0    -1
+$EndComp
+$Comp
+L 74xx:74LS04 U7
+U 3 1 5C0FE5B0
+P 6650 3900
+F 0 "U7" H 6650 4217 50  0000 C CNN
+F 1 "74LS04" H 6650 4126 50  0000 C CNN
+F 2 "" H 6650 3900 50  0001 C CNN
+F 3 "http://www.ti.com/lit/gpn/sn74LS04" H 6650 3900 50  0001 C CNN
+	3    6650 3900
+	1    0    0    -1
+$EndComp
+Wire Wire Line
+	6950 2750 7200 2750
+Wire Wire Line
+	7250 3900 6950 3900
 Wire Bus Line
 	10000 1750 10000 2050

Commit message: gerbers created, Rev 0 sent to manufacturer
Parts:
- U10: footprint (none) -> TO_SOT_Packages_THT:TO-92_Inline_Narrow_Oval
- U2, U8: footprint (none) -> Package_DIP:DIP-16_W7.62mm
- U7, U9: footprint (none) -> Package_DIP:DIP-14_W7.62mm
- X1, X2: footprint (none) -> Oscillator:Oscillator_DIP-14
Changed lines of the file:
@@
 F 0 "X2" H 6150 3750 50  0000 L CNN
 F 1 "8 MHZ" H 6100 3650 50  0000 L CNN
-F 2 "" H 6300 3550 50  0001 C CNN
+F 2 "Oscillator:Oscillator_DIP-14" H 6300 3550 50  0001 C CNN
 F 3 "http://cdn-reichelt.de/documents/datenblatt/B400/OSZI.pdf" H 5750 3900 50  0001 C CNN
 	1    5850 3900
@@
 F 0 "U2" H 3400 7878 50  0000 C CNN
 F 1 "74LS148" H 3400 7787 50  0000 C CNN
-F 2 "" H 3400 7000 50  0001 C CNN
+F 2 "Package_DIP:DIP-16_W7.62mm" H 3400 7000 50  0001 C CNN
 F 3 "http://www.ti.com/lit/gpn/sn74LS148" H 3400 7000 50  0001 C CNN
 	1    3400 7000
@@
 F 0 "U9" H 6800 6883 50  0000 C CNN
 F 1 "74LS10" H 6800 6974 50  0000 C CNN
-F 2 "" H 6800 7200 50  0001 C CNN
+F 2 "Package_DIP:DIP-14_W7.62mm" H 6800 7200 50  0001 C CNN
 F 3 "http://www.ti.com/lit/gpn/sn74LS10" H 6800 7200 50  0001 C CNN
 	1    6800 7200
@@
 F 0 "U8" H 5700 7678 50  0000 C CNN
 F 1 "74LS138" H 5700 7587 50  0000 C CNN
-F 2 "" H 5700 6900 50  0001 C CNN
+F 2 "Package_DIP:DIP-16_W7.62mm" H 5700 6900 50  0001 C CNN
 F 3 "http://www.ti.com/lit/gpn/sn74LS138" H 5700 6900 50  0001 C CNN
 	1    5700 6900
@@
 F 0 "U10" H 9070 4996 50  0000 R CNN
 F 1 "MCP100-485D" H 9070 4905 50  0000 R CNN
-F 2 "" H 8900 5100 50  0001 C CNN
+F 2 "TO_SOT_Packages_THT:TO-92_Inline_Narrow_Oval" H 8900 5100 50  0001 C CNN
 F 3 "http://ww1.microchip.com/downloads/en/DeviceDoc/11187f.pdf" H 9000 5200 50  0001 C CNN
 	1    9300 4950
@@
 F 0 "X1" H 6100 2600 50  0000 L CNN
 F 1 "3.6864 MHZ" H 6050 2500 50  0000 L CNN
-F 2 "" H 6250 2400 50  0001 C CNN
+F 2 "Oscillator:Oscillator_DIP-14" H 6250 2400 50  0001 C CNN
 F 3 "http://cdn-reichelt.de/documents/datenblatt/B400/OSZI.pdf" H 5700 2750 50  0001 C CNN
 	1    5800 2750
@@
 F 0 "U7" H 6200 1867 50  0000 C CNN
 F 1 "74LS04" H 6200 1776 50  0000 C CNN
-F 2 "" H 6200 1550 50  0001 C CNN
+F 2 "Package_DIP:DIP-14_W7.62mm" H 6200 1550 50  0001 C CNN
 F 3 "http://www.ti.com/lit/gpn/sn74LS04" H 6200 1550 50  0001 C CNN
 	1    6200 1550
@@
 F 0 "U7" H 6650 3067 50  0000 C CNN
 F 1 "74LS04" H 6650 2976 50  0000 C CNN
-F 2 "" H 6650 2750 50  0001 C CNN
+F 2 "Package_DIP:DIP-14_W7.62mm" H 6650 2750 50  0001 C CNN
 F 3 "http://www.ti.com/lit/gpn/sn74LS04" H 6650 2750 50  0001 C CNN
 	2    6650 2750
@@
 F 0 "U7" H 6650 4217 50  0000 C CNN
 F 1 "74LS04" H 6650 4126 50  0000 C CNN
-F 2 "" H 6650 3900 50  0001 C CNN
+F 2 "Package_DIP:DIP-14_W7.62mm" H 6650 3900 50  0001 C CNN
 F 3 "http://www.ti.com/lit/gpn/sn74LS04" H 6650 3900 50  0001 C CNN
 	3    6650 3900
