File: prototype/schematic/raven68k-proto/memdecode.sch (KiCad schematic (older format))
At the start: 8 parts

Commit message: breadboard prototype
Connections:
- net ~AS: now also U?.8 (CP)
Changed lines of the file:
@@
 Text GLabel 4350 4150 0    50   Input ~ 0
 SHADOW_RAM
-Text HLabel 4350 4600 0    50   Input ~ 0
-~AS
 $Comp
 L 74xx:74LS00 U?
@@
 Wire Wire Line
 	6550 4550 6650 4550
+Text HLabel 4350 4600 0    50   Input ~ 0
+~AS
+Wire Wire Line
+	2000 2650 1900 2650
 Wire Bus Line
 	1650 4100 1650 4400
+Text HLabel 1900 2650 0    50   Input ~ 0
+~AS
 $EndSCHEMATC

Commit message: optimizations
Parts:
- removed U? (x2): 74LS04, symbol 74xx:74LS04
- removed U?: 74LS00, symbol 74xx:74LS00
- added U2, U5: 74LS32, symbol 74xx:74LS32
- added unit 2 of U4
- added unit 3 of U4
- added U6: 74LS04, symbol 74xx:74LS04
- gave numbers to parts that had none: 5
Connections:
- net SHADOW_RAM: now also U2.1
- net ~AS: now also U2.2
- net ~DUART_CS: now also U2.5
- net ~RAM_CS: now also U2.13, U5.2
- net ~ROM_CS: now also U5.10, U5.5
- net ~RTC_CS: now also U2.10
- net at U4.1: now also U3.7 (O7)
- net ~ROMCS: no longer names the net of U4.2
- net ~ROMCS: now also U2.3; no longer U3.7 (O7)
- new net: U4.5, U4.9, U5.11
- new net: U4.6, U6.3
- new net: U4.10, U6.2
- new net: U4.8, U6.5
- new net R~W: U4.4, U6.1
- new net ~DUART_LCS: U2.6
- new net ~LDS: U2.12, U2.4, U2.9, U5.12, U5.4
- new net ~OE: U6.4
- new net ~RAM_LCS: U2.11
- new net ~RAM_UCS: U5.3
- new net ~ROM_LCS: U5.6
- new net ~ROM_UCS: U5.8
- new net ~RTC_LCS: U2.8
- new net ~UDS: U5.1, U5.13, U5.9
- new net ~WE: U6.6
Other:
- moved on the sheet: C2, U3, U4A
