File: rev1/schematic/raven68k-rev1/Interrupts.sch (KiCad schematic (older format))
At the start: 13 parts

Commit message: update schematic for rev1
Parts:
- removed C? (x3): 0.1uF, symbol Device:C_Small
- removed R?: 4.7k, symbol Device:R_Small
- removed U?: 74LS138, symbol 74xx:74LS138
- added C? (x2): 0.1uF, symbol Device:C
Connections:
- net +5V: now also C?.1, C?.1
- net GND: now also C?.2, C?.2
- net ~IACK_EN: now reaches U?.4 (E1)
- no-connect marks 10 -> 3
Other:
- note added: "IRQ7 does NOT need a pull-up\nas it is driven by SQW\n"

Commit message: added buffers
Parts:
- added U14: 74LS138, Package_DIP:DIP-16_W7.62mm, symbol 74xx:74LS138
- U8, U9: renamed from U?; footprint (none) -> Package_DIP:DIP-16_W7.62mm
- gave numbers to parts that had none: 8
Connections:
- net +5V: now also U14.16 (VCC), U14.6 (E3)
- net GND: now also U14.4 (E1), U14.5 (E2), U14.8 (GND)
- net ~IACK_EN: no longer names the net of U8.4 (E1)
- net ~IACK_EN: now also U14.7 (O7)
- new net FC0: U14.1 (A0)
- new net FC1: U14.2 (A1)
- new net FC2: U14.3 (A2)
- no-connect marks 3 -> 10
Other:
- moved on the sheet: C6, C7, R10, R11, R12, R7, R8, R9, U8, U9
