File: rev1/schematic/raven68k-rev1/Interrupts.sch (KiCad schematic (older format))
At the start: 11 parts, among them U14 74LS138, U8 74LS138, U9 74LS148

Commit message: upgrade to KiCad 6, first shot at layout
Parts:
- removed C6, C7: 0.1uF, symbol Device:C
- removed R10, R11, R12, R7, R8, R9: 4.7k, symbol Device:R_Small
- removed U14, U8: 74LS138, Package_DIP:DIP-16_W7.62mm, symbol 74xx:74LS138
- removed U9: 74LS148, Package_DIP:DIP-16_W7.62mm, symbol 74xx:74LS148
Connections:
- no-connect marks 10 -> 0
Other:
- note removed: "IRQ7 does NOT need a pull-up\nas it is driven by SQW\n"
