File: rev1/schematic/raven68k-rev1/power.sch (KiCad schematic (older format))
At the start: 33 parts, among them IC1 L5970D013TR, IC2 L5970D013TR, J3 Jack-DC

Commit message: upgrade to KiCad 6, first shot at layout
Parts:
- added D3: 3.3V, symbol Device:LED
- added F1: 2A, symbol Device:Fuse
- added R19: 330, symbol Device:R_Small
- added SW2: POWER_SW, symbol Switch:SW_SPST
- C12: renamed from C14; value 100nF -> 0.1uF; footprint (none) -> Capacitor_SMD:C_1206_3216Metric_Pad1.33x1.80mm_HandSolder
- C13: renamed from C15; value 100nF -> 0.1uF; footprint (none) -> Capacitor_SMD:C_1206_3216Metric_Pad1.33x1.80mm_HandSolder
- C14: renamed from C16; footprint (none) -> Capacitor_SMD:C_1206_3216Metric_Pad1.33x1.80mm_HandSolder
- C15: renamed from C17; footprint (none) -> Capacitor_SMD:C_1206_3216Metric_Pad1.33x1.80mm_HandSolder
- C16: renamed from C18; footprint (none) -> Capacitor_SMD:C_1206_3216Metric_Pad1.33x1.80mm_HandSolder
- C17: renamed from C19; footprint (none) -> Capacitor_SMD:C_1206_3216Metric_Pad1.33x1.80mm_HandSolder
- C18: renamed from C20; footprint (none) -> Capacitor_SMD:C_1206_3216Metric_Pad1.33x1.80mm_HandSolder
- C19: renamed from C21; footprint (none) -> Capacitor_SMD:C_1206_3216Metric_Pad1.33x1.80mm_HandSolder
- C20: renamed from C22; footprint (none) -> Capacitor_SMD:C_1206_3216Metric_Pad1.33x1.80mm_HandSolder
- C21: renamed from C23; footprint (none) -> Capacitor_SMD:C_1206_3216Metric_Pad1.33x1.80mm_HandSolder
- C22: renamed from C24; footprint (none) -> Capacitor_SMD:C_1206_3216Metric_Pad1.33x1.80mm_HandSolder
- C23: renamed from C25; footprint (none) -> Capacitor_SMD:C_1206_3216Metric_Pad1.33x1.80mm_HandSolder
- C24: renamed from C26; footprint (none) -> Capacitor_SMD:C_1206_3216Metric_Pad1.33x1.80mm_HandSolder
- C25: renamed from C27; footprint (none) -> Capacitor_SMD:C_1206_3216Metric_Pad1.33x1.80mm_HandSolder
- C26: renamed from C28; footprint (none) -> Capacitor_SMD:C_1206_3216Metric_Pad1.33x1.80mm_HandSolder
- C27: renamed from C29; footprint (none) -> Capacitor_SMD:C_1206_3216Metric_Pad1.33x1.80mm_HandSolder
- D1, D2: footprint Diode_THT:D_DO-41_SOD81_P10.16mm_Horizontal -> (none)
- D4: renamed from D3; value LED -> 5V
- IC1, IC2: footprint SOIC127P600X175-8N -> (none)
- L1, L2: footprint SRN5040TA101K -> (none)
- renumbered R21 to R11, R22 to R12, R23 to R13, R24 to R14, R25 to R15, R26 to R16, R27 to R17, R28 to R18, R29 to R20
Connections:
- net +3V3: now also R19.1
- net at C12.1, C13.1, C14.1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: now also D3.1 (K)
- net at C12.2, C13.2, C14.2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: now also F1.1; no longer J3.1
- new net: J3.1, SW2.1 (A)
- new net: D3.2 (A), R19.2
- new net: F1.2, SW2.2 (B)
Other:
- moved on the sheet: C12, C13, C14, C15, C16, C17, C18, C19, C20, C21, C22, C23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
