File: rev1/schematic/raven68k-rev1/ram-rom.sch (KiCad schematic (older format))
At the start: 8 parts, among them U10 KM684000BLP-7L, U11 KM684000BLP-7L, U12 28C256, U13 28C256

Commit message: upgrade to KiCad 6, first shot at layout
Parts:
- C10, C11, C8, C9: footprint (none) -> Capacitor_SMD:C_1206_3216Metric_Pad1.33x1.80mm_HandSolder
- U10: renamed from U12; footprint Package_DIP:DIP-28_W7.62mm_Socket -> Package_DIP:DIP-28_W15.24mm_Socket_LongPads
- U11: renamed from U13; footprint Package_DIP:DIP-28_W7.62mm_Socket -> Package_DIP:DIP-28_W15.24mm_Socket_LongPads
- U8: renamed from U10; footprint Package_DIP:DIP-32_W15.24mm -> Package_DIP:DIP-32_W15.24mm_Socket_LongPads
- U9: renamed from U11; footprint Package_DIP:DIP-32_W15.24mm -> Package_DIP:DIP-32_W15.24mm_Socket_LongPads
Changed lines of the file:
@@
 $Descr A4 11693 8268
 encoding utf-8
-Sheet 4 6
+Sheet 3 5
 Title ""
 Date ""
@@
 $EndDescr
 $Comp
-L custom:KM684000BLP-7L U11
+L custom:KM684000BLP-7L U9
 U 1 1 60787FA0
 P 2500 2500
-F 0 "U11" H 2500 3781 50  0000 C CNN
+F 0 "U9" H 2500 3781 50  0000 C CNN
 F 1 "KM684000BLP-7L" H 2500 3690 50  0000 C CNN
-F 2 "Package_DIP:DIP-32_W15.24mm" H 2500 2600 50  0001 C CNN
+F 2 "Package_DIP:DIP-32_W15.24mm_Socket_LongPads" H 2500 2600 50  0001 C CNN
 F 3 "https://pdf1.alldatasheet.com/datasheet-pdf/view/37316/SAMSUNG/KM684000BLP-7L/+25_2JUOYlSuOpdxSw.wYvzMXdxLb+/datasheet.pdf" H 2500 2600 50  0001 C CNN
 	1    2500 2500
@@
 $EndComp
 $Comp
-L custom:KM684000BLP-7L U10
+L custom:KM684000BLP-7L U8
 U 1 1 60788BE7
 P 2450 5250
-F 0 "U10" H 2450 6531 50  0000 C CNN
+F 0 "U8" H 2450 6531 50  0000 C CNN
 F 1 "KM684000BLP-7L" H 2450 6440 50  0000 C CNN
-F 2 "Package_DIP:DIP-32_W15.24mm" H 2450 5350 50  0001 C CNN
+F 2 "Package_DIP:DIP-32_W15.24mm_Socket_LongPads" H 2450 5350 50  0001 C CNN
 F 3 "https://pdf1.alldatasheet.com/datasheet-pdf/view/37316/SAMSUNG/KM684000BLP-7L/+25_2JUOYlSuOpdxSw.wYvzMXdxLb+/datasheet.pdf" H 2450 5350 50  0001 C CNN
 	1    2450 5250
@@
 $EndComp
 $Comp
-L Memory_EEPROM:28C256 U12
+L Memory_EEPROM:28C256 U10
 U 1 1 6078A07C
 P 6450 2400
-F 0 "U12" H 6450 3681 50  0000 C CNN
+F 0 "U10" H 6450 3681 50  0000 C CNN
 F 1 "28C256" H 6450 3590 50  0000 C CNN
-F 2 "Package_DIP:DIP-28_W7.62mm_Socket" H 6450 2400 50  0001 C CNN
+F 2 "Package_DIP:DIP-28_W15.24mm_Socket_LongPads" H 6450 2400 50  0001 C CNN
 F 3 "http://ww1.microchip.com/downloads/en/DeviceDoc/doc0006.pdf" H 6450 2400 50  0001 C CNN
 	1    6450 2400
@@
 Wire Wire Line
 	6050 1500 5900 1500
-Wire Wire Line
-	6050 1600 5900 1600
 Wire Wire Line
 	6050 1700 5900 1700
@@
 Text HLabel 5900 5950 0    50   Input ~ 0
 ~OE
-Text Label 5900 1500 0    50   ~ 0
+Text Label 5950 1500 0    50   ~ 0
 A1
-Text Label 5900 1600 0    50   ~ 0
+Text Label 5950 1600 0    50   ~ 0
 A2
-Text Label 5900 1700 0    50   ~ 0
+Text Label 5950 1700 0    50   ~ 0
 A3
-Text Label 5900 1800 0    50   ~ 0
+Text Label 5950 1800 0    50   ~ 0
 A4
-Text Label 5900 1900 0    50   ~ 0
+Text Label 5950 1900 0    50   ~ 0
 A5
-Text Label 5900 2000 0    50   ~ 0
+Text Label 5950 2000 0    50   ~ 0
 A6
-Text Label 5900 2100 0    50   ~ 0
+Text Label 5950 2100 0    50   ~ 0
 A7
-Text Label 5900 2200 0    50   ~ 0
+Text Label 5950 2200 0    50   ~ 0
 A8
-Text Label 5900 2300 0    50   ~ 0
+Text Label 5950 2300 0    50   ~ 0
 A9
-Text Label 5900 2400 0    50   ~ 0
+Text Label 5950 2400 0    50   ~ 0
 A10
-Text Label 5900 2500 0    50   ~ 0
+Text Label 5950 2500 0    50   ~ 0
 A11
-Text Label 5900 2600 0    50   ~ 0
+Text Label 5950 2600 0    50   ~ 0
 A12
-Text Label 5900 2700 0    50   ~ 0
+Text Label 5950 2700 0    50   ~ 0
 A13
-Text Label 5900 2800 0    50   ~ 0
+Text Label 5950 2800 0    50   ~ 0
 A14
-Text Label 5900 2900 0    50   ~ 0
+Text Label 5950 2900 0    50   ~ 0
 A15
 Text Label 5900 4250 0    50   ~ 0
@@
 Wire Wire Line
 	1800 1700 2000 1700
-Wire Wire Line
-	1800 1800 2000 1800
 Wire Wire Line
 	1800 1900 2000 1900
@@
 F 0 "C8" H 3815 7096 50  0000 L CNN
 F 1 "0.1uF" H 3815 7005 50  0000 L CNN
-F 2 "" H 3738 6900 50  0001 C CNN
+F 2 "Capacitor_SMD:C_1206_3216Metric_Pad1.33x1.80mm_HandSolder" H 3738 6900 50  0001 C CNN
 F 3 "~" H 3700 7050 50  0001 C CNN
 	1    3700 7050
@@
 AR Path="/610A1F9D/6201DDD0" Ref="#PWR?"  Part="1"
 AR Path="/60A4B12C/6201DDD0" Ref="#PWR?"  Part="1"
-AR Path="/6077E967/6201DDD0" Ref="#PWR044"  Part="1"
-F 0 "#PWR044" H 3100 7200 50  0001 C CNN
+AR Path="/6077E967/6201DDD0" Ref="#PWR041"  Part="1"
+F 0 "#PWR041" H 3100 7200 50  0001 C CNN
 F 1 "GND" H 3105 7277 50  0000 C CNN
 F 2 "" H 3100 7450 50  0001 C CNN
@@
 AR Path="/610A1F9D/6201DDD6" Ref="#PWR?"  Part="1"
 AR Path="/60A4B12C/6201DDD6" Ref="#PWR?"  Part="1"
-AR Path="/6077E967/6201DDD6" Ref="#PWR043"  Part="1"
-F 0 "#PWR043" H 3100 6550 50  0001 C CNN
+AR Path="/6077E967/6201DDD6" Ref="#PWR040"  Part="1"
+F 0 "#PWR040" H 3100 6550 50  0001 C CNN
 F 1 "+5V" H 3115 6873 50  0000 C CNN
 F 2 "" H 3100 6700 50  0001 C CNN
@@
 F 0 "C9" H 4265 7096 50  0000 L CNN
 F 1 "0.1uF" H 4265 7005 50  0000 L CNN
-F 2 "" H 4188 6900 50  0001 C CNN
+F 2 "Capacitor_SMD:C_1206_3216Metric_Pad1.33x1.80mm_HandSolder" H 4188 6900 50  0001 C CNN
 F 3 "~" H 4150 7050 50  0001 C CNN
 	1    4150 7050
@@
 F 0 "C10" H 4715 7096 50  0000 L CNN
 F 1 "0.1uF" H 4715 7005 50  0000 L CNN
-F 2 "" H 4638 6900 50  0001 C CNN
+F 2 "Capacitor_SMD:C_1206_3216Metric_Pad1.33x1.80mm_HandSolder" H 4638 6900 50  0001 C CNN
 F 3 "~" H 4600 7050 50  0001 C CNN
 	1    4600 7050
@@
 F 0 "C11" H 5165 7096 50  0000 L CNN
 F 1 "0.1uF" H 5165 7005 50  0000 L CNN
-F 2 "" H 5088 6900 50  0001 C CNN
+F 2 "Capacitor_SMD:C_1206_3216Metric_Pad1.33x1.80mm_HandSolder" H 5088 6900 50  0001 C CNN
 F 3 "~" H 5050 7050 50  0001 C CNN
 	1    5050 7050
@@
 Odd
 $Comp
-L Memory_EEPROM:28C256 U13
+L Memory_EEPROM:28C256 U11
 U 1 1 6078A57A
 P 6450 5150
-F 0 "U13" H 6450 6431 50  0000 C CNN
+F 0 "U11" H 6450 6431 50  0000 C CNN
 F 1 "28C256" H 6450 6340 50  0000 C CNN
-F 2 "Package_DIP:DIP-28_W7.62mm_Socket" H 6450 5150 50  0001 C CNN
+F 2 "Package_DIP:DIP-28_W15.24mm_Socket_LongPads" H 6450 5150 50  0001 C CNN
 F 3 "http://ww1.microchip.com/downloads/en/DeviceDoc/doc0006.pdf" H 6450 5150 50  0001 C CNN
 	1    6450 5150
@@
 AR Path="/610A1F9D/625AA722" Ref="#PWR?"  Part="1"
 AR Path="/60A4B12C/625AA722" Ref="#PWR?"  Part="1"
-AR Path="/6077E967/625AA722" Ref="#PWR039"  Part="1"
-F 0 "#PWR039" H 2550 6100 50  0001 C CNN
+AR Path="/6077E967/625AA722" Ref="#PWR036"  Part="1"
+F 0 "#PWR036" H 2550 6100 50  0001 C CNN
 F 1 "GND" H 2555 6177 50  0000 C CNN
 F 2 "" H 2550 6350 50  0001 C CNN
@@
 AR Path="/610A1F9D/625AAAB7" Ref="#PWR?"  Part="1"
 AR Path="/60A4B12C/625AAAB7" Ref="#PWR?"  Part="1"
-AR Path="/6077E967/625AAAB7" Ref="#PWR048"  Part="1"
-F 0 "#PWR048" H 6550 6000 50  0001 C CNN
+AR Path="/6077E967/625AAAB7" Ref="#PWR045"  Part="1"
+F 0 "#PWR045" H 6550 6000 50  0001 C CNN
 F 1 "GND" H 6555 6077 50  0000 C CNN
 F 2 "" H 6550 6250 50  0001 C CNN
@@
 AR Path="/610A1F9D/625B185E" Ref="#PWR?"  Part="1"
 AR Path="/60A4B12C/625B185E" Ref="#PWR?"  Part="1"
-AR Path="/6077E967/625B185E" Ref="#PWR047"  Part="1"
-F 0 "#PWR047" H 6550 3250 50  0001 C CNN
+AR Path="/6077E967/625B185E" Ref="#PWR044"  Part="1"
+F 0 "#PWR044" H 6550 3250 50  0001 C CNN
 F 1 "GND" H 6555 3327 50  0000 C CNN
 F 2 "" H 6550 3500 50  0001 C CNN
@@
 AR Path="/610A1F9D/625B1C0A" Ref="#PWR?"  Part="1"
 AR Path="/60A4B12C/625B1C0A" Ref="#PWR?"  Part="1"
-AR Path="/6077E967/625B1C0A" Ref="#PWR040"  Part="1"
-F 0 "#PWR040" H 2600 3350 50  0001 C CNN
+AR Path="/6077E967/625B1C0A" Ref="#PWR037"  Part="1"
+F 0 "#PWR037" H 2600 3350 50  0001 C CNN
 F 1 "GND" H 2605 3427 50  0000 C CNN
 F 2 "" H 2600 3600 50  0001 C CNN
@@
 AR Path="/610A1F9D/625B2B6F" Ref="#PWR?"  Part="1"
 AR Path="/60A4B12C/625B2B6F" Ref="#PWR?"  Part="1"
-AR Path="/6077E967/625B2B6F" Ref="#PWR046"  Part="1"
-F 0 "#PWR046" H 5650 5700 50  0001 C CNN
+AR Path="/6077E967/625B2B6F" Ref="#PWR043"  Part="1"
+F 0 "#PWR043" H 5650 5700 50  0001 C CNN
 F 1 "+5V" H 5665 6023 50  0000 C CNN
 F 2 "" H 5650 5850 50  0001 C CNN
@@
 AR Path="/610A1F9D/625B3181" Ref="#PWR?"  Part="1"
 AR Path="/60A4B12C/625B3181" Ref="#PWR?"  Part="1"
-AR Path="/6077E967/625B3181" Ref="#PWR045"  Part="1"
-F 0 "#PWR045" H 5400 2950 50  0001 C CNN
+AR Path="/6077E967/625B3181" Ref="#PWR042"  Part="1"
+F 0 "#PWR042" H 5400 2950 50  0001 C CNN
 F 1 "+5V" H 5415 3273 50  0000 C CNN
 F 2 "" H 5400 3100 50  0001 C CNN
@@
 AR Path="/610A1F9D/625CA938" Ref="#PWR?"  Part="1"
 AR Path="/60A4B12C/625CA938" Ref="#PWR?"  Part="1"
-AR Path="/6077E967/625CA938" Ref="#PWR050"  Part="1"
-F 0 "#PWR050" H 6800 3900 50  0001 C CNN
+AR Path="/6077E967/625CA938" Ref="#PWR047"  Part="1"
+F 0 "#PWR047" H 6800 3900 50  0001 C CNN
 F 1 "+5V" H 6815 4223 50  0000 C CNN
 F 2 "" H 6800 4050 50  0001 C CNN
@@
 AR Path="/610A1F9D/625CAF84" Ref="#PWR?"  Part="1"
 AR Path="/60A4B12C/625CAF84" Ref="#PWR?"  Part="1"
-AR Path="/6077E967/625CAF84" Ref="#PWR049"  Part="1"
-F 0 "#PWR049" H 6800 1150 50  0001 C CNN
+AR Path="/6077E967/625CAF84" Ref="#PWR046"  Part="1"
+F 0 "#PWR046" H 6800 1150 50  0001 C CNN
 F 1 "+5V" H 6815 1473 50  0000 C CNN
 F 2 "" H 6800 1300 50  0001 C CNN
@@
 AR Path="/610A1F9D/625CB58A" Ref="#PWR?"  Part="1"
 AR Path="/60A4B12C/625CB58A" Ref="#PWR?"  Part="1"
-AR Path="/6077E967/625CB58A" Ref="#PWR042"  Part="1"
-F 0 "#PWR042" H 2950 1250 50  0001 C CNN
+AR Path="/6077E967/625CB58A" Ref="#PWR039"  Part="1"
+F 0 "#PWR039" H 2950 1250 50  0001 C CNN
 F 1 "+5V" H 2965 1573 50  0000 C CNN
 F 2 "" H 2950 1400 50  0001 C CNN
@@
 AR Path="/610A1F9D/625CBA19" Ref="#PWR?"  Part="1"
 AR Path="/60A4B12C/625CBA19" Ref="#PWR?"  Part="1"
-AR Path="/6077E967/625CBA19" Ref="#PWR041"  Part="1"
-F 0 "#PWR041" H 2900 4000 50  0001 C CNN
+AR Path="/6077E967/625CBA19" Ref="#PWR038"  Part="1"
+F 0 "#PWR038" H 2900 4000 50  0001 C CNN
 F 1 "+5V" H 2915 4323 50  0000 C CNN
 F 2 "" H 2900 4150 50  0001 C CNN
@@
 	1    0    0    -1
 $EndComp
+Wire Wire Line
+	3100 6850 3700 6850
+Wire Wire Line
+	3100 7300 3700 7300
+Wire Wire Line
+	1800 1800 2000 1800
+Wire Wire Line
+	6050 1600 5900 1600
 Wire Bus Line
 	7100 3800 7100 5050
@@
 Wire Bus Line
 	1700 800  1700 6250
-Wire Wire Line
-	3100 6850 3700 6850
-Wire Wire Line
-	3100 7300 3700 7300
 $EndSCHEMATC
