File: rev1/schematic/raven68k-rev1/ram-rom.kicad_sch (KiCad schematic)
At the start: 8 parts, among them U10 28C256, U11 28C256, U8 KM684000BLP-7L, U9 KM684000BLP-7L

Commit message: some helpful labels
Parts:
- C10, C11, C8, C9: LCSC (none) -> C24497
Changed lines of the file:
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@@
+      (effects (font (size 1.27 1.27)) hide)
+    )
+    (property "LCSC" "C24497" (id 4) (at 93.98 179.07 0)
       (effects (font (size 1.27 1.27)) hide)
     )
@@
       (effects (font (size 1.27 1.27)) hide)
     )
+    (property "LCSC" "C24497" (id 4) (at 105.41 179.07 0)
+      (effects (font (size 1.27 1.27)) hide)
+    )
     (pin "1")
     (pin "2")
@@
     )
     (property "Datasheet" "~" (id 3) (at 116.84 179.07 0)
+      (effects (font (size 1.27 1.27)) hide)
+    )
+    (property "LCSC" "C24497" (id 4) (at 116.84 179.07 0)
       (effects (font (size 1.27 1.27)) hide)
     )
@@
       (effects (font (size 1.27 1.27)) hide)
     )
+    (property "LCSC" "C24497" (id 4) (at 128.27 179.07 0)
+      (effects (font (size 1.27 1.27)) hide)
+    )
