File: rev1/schematic/raven68k-rev1/raven68k-rev1.kicad_pcb (KiCad board)
At the start: 2 copper layers, 196.8 x 123.2 mm, 16 parts, among them J1 CPLD_JTAG, U1 MCP100-485D, U10 KM684000BLP-7L, U11 KM684000BLP-7L, U12 28C256, U13 28C256, U2 68010D, U3 XC9572XL-VQ44, U4 68681, U5 74LS373, U6 CONSOLE, U7 DS12887+, U8 74LS138, U9 74LS148, X1 CLOCK, X2 CXO_DIP14

Commit message: upgrade to KiCad 6, first shot at layout
Parts:
- removed U12, U13: 28C256, Package_DIP:DIP-28_W7.62mm_Socket
- added C1: 0.1uF, Capacitor_SMD:C_1206_3216Metric_Pad1.33x1.80mm_HandSolder, B.Cu at (44.5, 78.7)
- added C10: 0.1uF, Capacitor_SMD:C_1206_3216Metric_Pad1.33x1.80mm_HandSolder, B.Cu at (138.4, 96.5)
- added C11: 0.1uF, Capacitor_SMD:C_1206_3216Metric_Pad1.33x1.80mm_HandSolder, B.Cu at (138.5, 50.8)
- added C12: 0.1uF, Capacitor_SMD:C_1206_3216Metric_Pad1.33x1.80mm_HandSolder, F.Cu at (214.6, 47.0)
- added C13: 0.1uF, Capacitor_SMD:C_1206_3216Metric_Pad1.33x1.80mm_HandSolder, F.Cu at (214.6, 66.0)
- added C14: 10uF, Capacitor_SMD:C_1206_3216Metric_Pad1.33x1.80mm_HandSolder, F.Cu at (210.8, 47.0)
- added C15: 10uF, Capacitor_SMD:C_1206_3216Metric_Pad1.33x1.80mm_HandSolder, F.Cu at (210.8, 66.0)
- added C16: 220pF, Capacitor_SMD:C_1206_3216Metric_Pad1.33x1.80mm_HandSolder, F.Cu at (207.0, 47.0)
- added C17: 220pF, Capacitor_SMD:C_1206_3216Metric_Pad1.33x1.80mm_HandSolder, F.Cu at (207.0, 66.0)
- added C18: 22nF, Capacitor_SMD:C_1206_3216Metric_Pad1.33x1.80mm_HandSolder, F.Cu at (201.9, 47.0)
- added C19: 22nF, Capacitor_SMD:C_1206_3216Metric_Pad1.33x1.80mm_HandSolder, F.Cu at (201.9, 66.0)
- added C2: 0.1uF, Capacitor_SMD:C_1206_3216Metric_Pad1.33x1.80mm_HandSolder, B.Cu at (80.0, 83.8)
- added C20: 470pF, Capacitor_SMD:C_1206_3216Metric_Pad1.33x1.80mm_HandSolder, F.Cu at (185.4, 45.7)
- added C21: 470pF, Capacitor_SMD:C_1206_3216Metric_Pad1.33x1.80mm_HandSolder, F.Cu at (185.4, 64.8)
- added C22: 47uF, Capacitor_SMD:C_1206_3216Metric_Pad1.33x1.80mm_HandSolder, F.Cu at (181.6, 41.9)
- added C23: 47uF, Capacitor_SMD:C_1206_3216Metric_Pad1.33x1.80mm_HandSolder, F.Cu at (181.6, 61.0)
- added C24: 47uF, Capacitor_SMD:C_1206_3216Metric_Pad1.33x1.80mm_HandSolder, F.Cu at (177.8, 41.9)
- added C25: 47uF, Capacitor_SMD:C_1206_3216Metric_Pad1.33x1.80mm_HandSolder, F.Cu at (177.8, 61.0)
- added C26: 100nF, Capacitor_SMD:C_1206_3216Metric_Pad1.33x1.80mm_HandSolder, F.Cu at (174.0, 41.9)
- added C27: 100nF, Capacitor_SMD:C_1206_3216Metric_Pad1.33x1.80mm_HandSolder, F.Cu at (174.0, 61.0)
- added C3: 0.1uF, Capacitor_SMD:C_1206_3216Metric_Pad1.33x1.80mm_HandSolder, F.Cu at (85.1, 132.1)
- added C4: 0.1uF, Capacitor_SMD:C_1206_3216Metric_Pad1.33x1.80mm_HandSolder, F.Cu at (81.3, 132.1)
- added C5: 0.1uF, Capacitor_SMD:C_1206_3216Metric_Pad1.33x1.80mm_HandSolder, B.Cu at (176.5, 81.3)
- added C6: 0.1uF, Capacitor_SMD:C_1206_3216Metric_Pad1.33x1.80mm_HandSolder, B.Cu at (203.2, 85.1)
- added C7: 0.1uF, Capacitor_SMD:C_1206_3216Metric_Pad1.33x1.80mm_HandSolder, B.Cu at (204.5, 114.3)
- added C8: 0.1uF, Capacitor_SMD:C_1206_3216Metric_Pad1.33x1.80mm_HandSolder, B.Cu at (110.2, 91.4)
- added C9: 0.1uF, Capacitor_SMD:C_1206_3216Metric_Pad1.33x1.80mm_HandSolder, B.Cu at (110.5, 45.7)
- added D1: SB140, Diode_SMD:D_1206_3216Metric_Pad1.42x1.75mm_HandSolder, F.Cu at (195.6, 49.5)
- added D2: SB140, Diode_SMD:D_1206_3216Metric_Pad1.42x1.75mm_HandSolder, F.Cu at (195.6, 68.6)
- added D3: 3.3V, LED_THT:LED_D3.0mm, F.Cu at (177.8, 55.9)
- added D4: 5V, LED_THT:LED_D3.0mm, F.Cu at (177.8, 47.0)
- added D5: LED, LED_THT:LED_D3.0mm, F.Cu at (223.5, 102.9)
- added H1: IDE-44-PIN, raven68k-rev1:SHDR44W55P200_2X22_4665X630X640P, F.Cu at (231.4, 65.4)
- added IC1: L5970D013TR, Package_SO:SO-8_5.3x6.2mm_P1.27mm, F.Cu at (198.1, 54.6)
- added IC2: L5970D013TR, Package_SO:SO-8_5.3x6.2mm_P1.27mm, F.Cu at (198.1, 73.7)
- added J2: DUART_IO, Connector_PinHeader_2.54mm:PinHeader_2x08_P2.54mm_Vertical, F.Cu at (231.1, 116.8)
- added J3: Jack-DC, raven68k-rev1:RAPC722BK, F.Cu at (235.0, 53.8)
- added L1: SRN5040TA-101K, raven68k-rev1:SRN5040TA101K, F.Cu at (195.6, 43.2)
- added L2: SRN5040TA-101K, raven68k-rev1:SRN5040TA101K, F.Cu at (195.6, 62.2)
- added R1: 2.2k, Resistor_SMD:R_1206_3216Metric_Pad1.30x1.75mm_HandSolder, B.Cu at (44.5, 73.7)
- added R10: 10K, Resistor_SMD:R_1206_3216Metric_Pad1.30x1.75mm_HandSolder, B.Cu at (226.1, 94.0)
- added R11: 4.7K, Resistor_SMD:R_1206_3216Metric_Pad1.30x1.75mm_HandSolder, F.Cu at (203.2, 41.9)
- added R12: 4.7K, Resistor_SMD:R_1206_3216Metric_Pad1.30x1.75mm_HandSolder, F.Cu at (203.2, 61.0)
- added R13: 3.9K, Resistor_SMD:R_1206_3216Metric_Pad1.30x1.75mm_HandSolder, F.Cu at (189.2, 41.9)
- added R14: 1.2K, Resistor_SMD:R_1206_3216Metric_Pad1.30x1.75mm_HandSolder, F.Cu at (189.2, 49.5)
- added R15: 4.7K, Resistor_SMD:R_1206_3216Metric_Pad1.30x1.75mm_HandSolder, F.Cu at (189.2, 61.0)
- added R16: 2.7K, Resistor_SMD:R_1206_3216Metric_Pad1.30x1.75mm_HandSolder, F.Cu at (189.2, 68.6)
- added R17: 390, Resistor_SMD:R_1206_3216Metric_Pad1.30x1.75mm_HandSolder, F.Cu at (185.4, 41.9)
- added R18: 390, Resistor_SMD:R_1206_3216Metric_Pad1.30x1.75mm_HandSolder, F.Cu at (185.4, 61.0)
- added R19: 330, Resistor_SMD:R_1206_3216Metric_Pad1.30x1.75mm_HandSolder, F.Cu at (174.0, 54.6)
- added R2: 2.2k, Resistor_SMD:R_1206_3216Metric_Pad1.30x1.75mm_HandSolder, B.Cu at (44.5, 71.1)
- added R20: 680, Resistor_SMD:R_1206_3216Metric_Pad1.30x1.75mm_HandSolder, F.Cu at (174.0, 48.3)
- added R21: 680, Resistor_SMD:R_1206_3216Metric_Pad1.30x1.75mm_HandSolder, B.Cu at (222.2, 106.7)
- added R3: 2.2k, Resistor_SMD:R_1206_3216Metric_Pad1.30x1.75mm_HandSolder, B.Cu at (44.5, 76.2)
- added R4: 2.2k, Resistor_SMD:R_1206_3216Metric_Pad1.30x1.75mm_HandSolder, B.Cu at (44.5, 96.5)
- added R5: 2.2k, Resistor_SMD:R_1206_3216Metric_Pad1.30x1.75mm_HandSolder, B.Cu at (44.5, 99.1)
- added R6: 4.7k, Resistor_SMD:R_1206_3216Metric_Pad1.30x1.75mm_HandSolder, B.Cu at (139.7, 101.6)
- added R7: 4.7k, Resistor_SMD:R_1206_3216Metric_Pad1.30x1.75mm_HandSolder, B.Cu at (176.5, 129.5)
- added R8: 4.7k, Resistor_SMD:R_1206_3216Metric_Pad1.30x1.75mm_HandSolder, B.Cu at (204.5, 127.0)
- added R9: 10K, Resistor_SMD:R_1206_3216Metric_Pad1.30x1.75mm_HandSolder, B.Cu at (226.1, 85.1)
- added RN1: 22, Package_DIP:DIP-16_W7.62mm_Socket_LongPads, F.Cu at (212.1, 78.7)
- added SW1: RESET_SW, raven68k-rev1:TS0266170BK160SCRD, F.Cu at (159.3, 47.3)
- added SW2: POWER_SW, raven68k-rev1:10TC605, F.Cu at (222.2, 47.0)
- U1: value MCP100-485D -> MCP100-465D; footprint Package_TO_SOT_THT:TO-92L_Inline_Wide -> Package_TO_SOT_THT:TO-92L_HandSolder
- U10, U11: value KM684000BLP-7L -> 28C256; footprint Package_DIP:DIP-32_W15.24mm -> Package_DIP:DIP-28_W15.24mm_Socket_LongPads
- U2: footprint Package_DIP:DIP-64_W25.4mm_Socket -> Package_DIP:DIP-64_W25.4mm_Socket_LongPads
- U4: footprint Package_DIP:DIP-40_W25.4mm_Socket -> Package_DIP:DIP-40_W25.4mm_Socket_LongPads
- U5: footprint Package_DIP:DIP-20_W7.62mm -> Package_DIP:DIP-20_W7.62mm_Socket_LongPads
- U6: footprint Connector_PinHeader_1.00mm:PinHeader_1x06_P1.00mm_Vertical -> Connector_PinHeader_2.54mm:PinHeader_1x06_P2.54mm_Vertical
- U7: footprint Package_DIP:DIP-24_W7.62mm -> Package_DIP:DIP-24_W15.24mm_Socket_LongPads
- U8: value 74LS138 -> KM684000BLP-7L; footprint Package_DIP:DIP-16_W7.62mm -> Package_DIP:DIP-32_W15.24mm_Socket_LongPads
- U9: value 74LS148 -> KM684000BLP-7L; footprint Package_DIP:DIP-16_W7.62mm -> Package_DIP:DIP-32_W15.24mm_Socket_LongPads
- X1, X2: footprint Oscillator:Oscillator_DIP-14 -> Oscillator:Oscillator_DIP-14_LargePads
- moved X1 161.6 mm to (54.6, 141.0)
- moved U1 146.0 mm to (162.6, 41.9)
- moved U9 139.2 mm to (88.9, 45.7)
- moved U11 129.9 mm to (116.8, 96.5)
- moved U6 121.2 mm to (152.4, 144.8), turned to 90 degrees
- moved U2 115.1 mm to (49.5, 45.7)
- moved U5 113.2 mm to (190.5, 85.1)
- moved U10 107.9 mm to (116.8, 50.8)
- moved U7 101.7 mm to (184.1, 114.3)
- moved X2 100.3 mm to (158.8, 59.7), turned to -90 degrees
- moved U8 98.3 mm to (88.9, 91.4)
- moved U4 91.6 mm to (146.1, 81.3)
- moved U3 88.1 mm to (92.7, 142.2), turned to 90 degrees
- moved J1 41.1 mm to (136.3, 45.1)
Connections:
- net R~W renamed R~{W}
- net ~CPU_DTACK renamed ~{CPU_DTACK}
- net ~DUART_CS renamed ~{DUART_CS}
- net ~LDS renamed ~{LDS}
- net ~RESET renamed ~{RESET}
- net ~UDS renamed ~{UDS}
- U10 pad 1: /RAM and ROM/A19 -> A15
- U10 pad 10: /RAM and ROM/A3 -> A1
- U10 pad 11: /RAM and ROM/A2 -> D8
- U10 pad 12: /RAM and ROM/A1 -> D9
- U10 pad 13: /RAM and ROM/D0 -> D10
- U10 pad 14: /RAM and ROM/D1 -> GND
- U10 pad 15: /RAM and ROM/D2 -> D11
- U10 pad 16: GND -> D12
- U10 pad 17: /RAM and ROM/D3 -> D13
- U10 pad 18: /RAM and ROM/D4 -> D14
- U10 pad 19: /RAM and ROM/D5 -> D15
- U10 pad 2: /RAM and ROM/A17 -> A13
- U10 pad 20: /RAM and ROM/D6 -> ~{ROM_UCE}
- U10 pad 21: /RAM and ROM/D7 -> A11
- U10 pad 22: ~RAM_LCE -> ~{OE}
- U10 pad 23: /RAM and ROM/A11 -> A12
- U10 pad 24: ~OE -> A10
- U10 pad 25: /RAM and ROM/A12 -> A9
- U10 pad 26: /RAM and ROM/A10 -> A14
- U10 pad 27: /RAM and ROM/A9 -> +5V
- U10 pad 28: /RAM and ROM/A14 -> +5V
- U10 pad 3: /RAM and ROM/A15 -> A8
- U10 pad 4: /RAM and ROM/A13 -> A7
- U10 pad 5: /RAM and ROM/A8 -> A6
- U10 pad 6: /RAM and ROM/A7 -> A5
- U10 pad 7: /RAM and ROM/A6 -> A4
- U10 pad 8: /RAM and ROM/A5 -> A3
- U10 pad 9: /RAM and ROM/A4 -> A2
- U11 pad 1: /RAM and ROM/A19 -> A15
- U11 pad 10: /RAM and ROM/A3 -> A1
- U11 pad 11: /RAM and ROM/A2 -> D0
- U11 pad 12: /RAM and ROM/A1 -> D1
- U11 pad 13: /RAM and ROM/D8 -> D2
- U11 pad 14: /RAM and ROM/D9 -> GND
- U11 pad 15: /RAM and ROM/D10 -> D3
- U11 pad 16: GND -> D4
- U11 pad 17: /RAM and ROM/D11 -> D5
- U11 pad 18: /RAM and ROM/D12 -> D6
- U11 pad 19: /RAM and ROM/D13 -> D7
- U11 pad 2: /RAM and ROM/A17 -> A13
- U11 pad 20: /RAM and ROM/D14 -> ~{ROM_LCE}
- U11 pad 21: /RAM and ROM/D15 -> A11
- U11 pad 22: ~RAM_UCE -> ~{OE}
- U11 pad 23: /RAM and ROM/A11 -> A12
- U11 pad 24: ~OE -> A10
- U11 pad 25: /RAM and ROM/A12 -> A9
- U11 pad 26: /RAM and ROM/A10 -> A14
- U11 pad 27: /RAM and ROM/A9 -> +5V
- U11 pad 28: /RAM and ROM/A14 -> +5V
- U11 pad 3: /RAM and ROM/A15 -> A8
- U11 pad 4: /RAM and ROM/A13 -> A7
- U11 pad 5: /RAM and ROM/A8 -> A6
- U11 pad 6: /RAM and ROM/A7 -> A5
- U11 pad 7: /RAM and ROM/A6 -> A4
- U11 pad 8: /RAM and ROM/A5 -> A3
- U11 pad 9: /RAM and ROM/A4 -> A2
- U2 pad 19: Net-(U2-Pad19) -> unconnected-(U2-Pad19)
- U2 pad 20: Net-(U2-Pad20) -> unconnected-(U2-Pad20)
- U2 pad 23: IPL2 -> ~{IPL2}
- U2 pad 24: IPL1 -> ~{IPL1}
- U2 pad 25: IPL0 -> ~{IPL0}
- U2 pad 6: ~AS -> ~{AS}
- U3 pad 1: Net-(U3-Pad1) -> unconnected-(U3-Pad1)
- U3 pad 15: +3V3 -> unconnected-(U3-Pad15)
- U3 pad 2: ~RTC_CE -> ~{RTC_CS}
- U3 pad 26: Net-(U3-Pad26) -> +3V3
- U3 pad 27: +5V -> ~{DUART_DTACK}
- U3 pad 28: ~IDE_CE2 -> ~{IDE_CS2}
- U3 pad 29: ~AS -> ~{AS}
- U3 pad 33: ~OE -> ~{OE}
- U3 pad 34: ~RAM_LCE -> ~{RAM_LCE}
- U3 pad 36: ~IDE_CE1 -> ~{IDE_CS1}
- U3 pad 37: ~RAM_UCE -> ~{RAM_UCE}
- U3 pad 38: ~ROM_LCE -> ~{ROM_LCE}
- U3 pad 39: ~ROM_UCE -> ~{ROM_UCE}
- U3 pad 40: Net-(U3-Pad40) -> FC0
- U3 pad 41: Net-(U3-Pad41) -> FC1
- U3 pad 42: Net-(U3-Pad42) -> FC2
- U3 pad 43: Net-(U3-Pad43) -> ~{DUART_IACK}
- U3 pad 44: Net-(U3-Pad44) -> unconnected-(U3-Pad44)
- U3 pad 6: ~OE -> ~{OE}
- U3 pad 7: ~AS -> ~{AS}
- U4 pad 1: /DUART and RTC/A1 -> A1
- U4 pad 16: /DUART and RTC/D1 -> D1
- U4 pad 17: /DUART and RTC/D3 -> D3
- U4 pad 18: /DUART and RTC/D5 -> D5
- U4 pad 19: /DUART and RTC/D7 -> D7
- U4 pad 21: ~DUART_IRQ -> ~{IPL0}
- U4 pad 22: /DUART and RTC/D6 -> D6
- U4 pad 23: /DUART and RTC/D4 -> D4
- U4 pad 24: /DUART and RTC/D2 -> D2
- U4 pad 25: /DUART and RTC/D0 -> D0
- U4 pad 3: /DUART and RTC/A2 -> A2
- U4 pad 30: TxDA -> RxDA
- U4 pad 31: RxDA -> TxDA
- U4 pad 33: Net-(U4-Pad33) -> unconnected-(U4-Pad33)
- U4 pad 37: ~DUART_IACK -> ~{DUART_IACK}
- U4 pad 5: /DUART and RTC/A3 -> A3
- U4 pad 6: /DUART and RTC/A4 -> A4
- U4 pad 9: Net-(R6-Pad1) -> ~{DUART_DTACK}
- U5 pad 12: /DUART and RTC/D4 -> D4
- U5 pad 13: /DUART and RTC/A5 -> A5
- U5 pad 14: /DUART and RTC/A6 -> A6
- U5 pad 15: /DUART and RTC/D5 -> D5
- U5 pad 16: /DUART and RTC/D6 -> D6
- U5 pad 17: /DUART and RTC/A7 -> A7
- U5 pad 18: /DUART and RTC/A8 -> A8
- U5 pad 19: /DUART and RTC/D7 -> D7
- U5 pad 2: /DUART and RTC/D0 -> D0
- U5 pad 3: /DUART and RTC/A1 -> A1
- U5 pad 4: /DUART and RTC/A2 -> A2
- U5 pad 5: /DUART and RTC/D1 -> D1
- U5 pad 6: /DUART and RTC/D2 -> D2
- U5 pad 7: /DUART and RTC/A3 -> A3
- U5 pad 8: /DUART and RTC/A4 -> A4
- U5 pad 9: /DUART and RTC/D3 -> D3
- U6 pad 1: Net-(U6-Pad1) -> unconnected-(U6-Pad1)
- U6 pad 5: Net-(U6-Pad5) -> unconnected-(U6-Pad5)
- U6 pad 6: Net-(U6-Pad6) -> unconnected-(U6-Pad6)
- U7 pad 10: /DUART and RTC/D6 -> D6
- U7 pad 11: /DUART and RTC/D7 -> D7
- U7 pad 13: ~RTC_CS -> ~{RTC_CS}
- U7 pad 19: ~RTC_IRQ -> ~{IPL1}
- U7 pad 23: SQU -> ~{IPL2}
- U7 pad 4: /DUART and RTC/D0 -> D0
- U7 pad 5: /DUART and RTC/D1 -> D1
- U7 pad 6: /DUART and RTC/D2 -> D2
- U7 pad 7: /DUART and RTC/D3 -> D3
- U7 pad 8: /DUART and RTC/D4 -> D4
- U7 pad 9: /DUART and RTC/D5 -> D5
- U8 pad 1: /Interrupts/A1 -> A19
- U8 pad 10: /Interrupts/~IACK5 -> A3
- U8 pad 11: /Interrupts/~IACK4 -> A2
- U8 pad 12: /Interrupts/~IACK3 -> A1
- U8 pad 13: /Interrupts/~IACK2 -> D0
- U8 pad 14: ~DUART_IACK -> D1
- U8 pad 15: Net-(U8-Pad15) -> D2
- U8 pad 16: +5V -> GND
- U8 pad 2: /Interrupts/A2 -> A17
- U8 pad 3: /Interrupts/A3 -> A15
- U8 pad 4: /Interrupts/~IACK_EN -> A13
- U8 pad 5: ~AS -> A8
- U8 pad 6: +5V -> A7
- U8 pad 7: /Interrupts/~IACK7 -> A6
- U8 pad 8: GND -> A5
- U8 pad 9: /Interrupts/~IACK6 -> A4
- U9 pad 1: /Interrupts/~IRQ4 -> A19
- U9 pad 10: GND -> A3
- U9 pad 11: ~DUART_IRQ -> A2
- U9 pad 12: ~RTC_IRQ -> A1
- U9 pad 13: ~IDE_IRQ -> D8
- U9 pad 14: Net-(U9-Pad14) -> D9
- U9 pad 15: Net-(U9-Pad15) -> D10
- U9 pad 16: +5V -> GND
- U9 pad 2: /Interrupts/~IRQ5 -> A17
- U9 pad 3: /Interrupts/~IRQ6 -> A15
- U9 pad 4: SQU -> A13
- U9 pad 5: GND -> A8
- U9 pad 6: /Interrupts/IPL2 -> A7
- U9 pad 7: /Interrupts/IPL1 -> A6
- U9 pad 8: GND -> A5
- U9 pad 9: /Interrupts/IPL0 -> A4
- X1 pad 1: Net-(X1-Pad1) -> unconnected-(X1-Pad1)
- X2 pad 1: Net-(X2-Pad1) -> unconnected-(X2-Pad1)
Routing:
- net +5V: track 0.00 -> 576.6 mm, vias 0 -> 1
- net +3V3: track 0.00 -> 184.9 mm
- net Net-(C12-Pad2): track 0.00 -> 93.7 mm
- net GND: track 0.00 -> 60.1 mm
- net Net-(C21-Pad2): track 0.00 -> 31.2 mm
- net Net-(C20-Pad2): track 0.00 -> 31.2 mm
- net Net-(J3-Pad1): track 0.00 -> 17.0 mm
- net Net-(IC1-Pad1): track 0.00 -> 11.1 mm
- net Net-(D2-Pad1): track 0.00 -> 8.24 mm
- net Net-(H1-Pad29): track 0.00 -> 4.06 mm
- net Net-(D4-Pad2): track 0.00 -> 3.93 mm
- net Net-(D3-Pad2): track 0.00 -> 3.93 mm
- net Net-(H1-Pad21): track 0.00 -> 3.91 mm
- net Net-(C19-Pad1): track 0.00 -> 3.63 mm
- net Net-(C18-Pad1): track 0.00 -> 3.63 mm
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Other:
- board size 196.8 x 123.2 mm -> 203.2 x 114.3 mm
- net class Default removed
- board text added: "CONSOLE"
- board text added: "EVEN"
- board text added: "JTAG"
- board text added: "ODD"

Commit message: board layout complete, needs verification
Parts:
- removed SW1: RESET_SW, raven68k-rev1:TS0266170BK160SCRD
- removed SW2: POWER_SW, raven68k-rev1:10TC605
- added S1: RESET_SW, raven68k-rev1:TS0266170BK160SCRD, F.Cu at (159.6, 48.7)
- added S2: POWER_SW, raven68k-rev1:GPTS203212B, F.Cu at (232.3, 45.7)
- C3, C4: moved to B.Cu
- J3: value Jack-DC -> RAPC722BK
- moved C4 90.5 mm to (142.5, 65.4), turned to 180 degrees
- moved U3 89.9 mm to (144.5, 68.8), turned to 180 degrees
- moved C3 84.4 mm to (144.5, 72.1), turned to 180 degrees
- moved J3 11.0 mm to (225.7, 59.7), turned to 90 degrees
- moved D5 5.08 mm to (223.5, 108.0)
- moved R21 5.08 mm to (222.2, 111.8)
- moved R9 4.96 mm to (226.3, 90.0)
- moved H1 4.86 mm to (233.1, 69.9)
- moved R10 3.82 mm to (226.3, 97.8)
- moved J2 1.69 mm to (232.8, 117.2)
Connections:
- J3 pad 1: Net-(J3-Pad1) -> VDD
- J3 pad 3: (no net) -> GND
Routing:
- net D3: track 0.00 -> 333.9 mm, vias 0 -> 3
- net A1: track 0.00 -> 323.5 mm, vias 0 -> 6
- net D5: track 0.00 -> 323.1 mm, vias 0 -> 4
- net A2: track 0.00 -> 316.2 mm, vias 0 -> 6
- net D2: track 0.00 -> 314.4 mm, vias 0 -> 2
- net D4: track 0.00 -> 313.7 mm, vias 0 -> 2
- net A3: track 0.00 -> 313.7 mm, vias 0 -> 4
- net D1: track 0.00 -> 312.6 mm
- net D0: track 0.00 -> 299.6 mm, vias 0 -> 1
- net D7: track 0.00 -> 299.1 mm, vias 0 -> 3
- net D6: track 0.00 -> 292.9 mm, vias 0 -> 6
- net A4: track 0.00 -> 267.4 mm, vias 0 -> 4
- net R~{W}: track 0.00 -> 256.4 mm, vias 0 -> 3
- net D8: track 0.00 -> 245.2 mm, vias 0 -> 2
- net ~{RESET}: track 0.00 -> 242.7 mm, vias 0 -> 3
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- added copper zone on B.Cu, net GND

Commit message: move components around
Parts:
- removed S1: RESET_SW, raven68k-rev1:TS0266170BK160SCRD
- added SW1: RESET_SW, raven68k-rev1:TS0266170BK160SCRD, F.Cu at (159.7, 48.9)
- C3, C4: moved to F.Cu
- moved J2 104.4 mm to (132.0, 144.3), turned to 90 degrees
- moved C11 82.8 mm to (55.8, 51.6), turned to 180 degrees
- moved C10 82.7 mm to (55.8, 97.2), turned to 180 degrees
- moved U10 71.5 mm to (45.3, 51.4)
- moved U11 71.5 mm to (45.3, 97.1)
- moved R5 62.4 mm to (106.8, 97.3), turned to 180 degrees
- moved C1 62.4 mm to (106.8, 77.1), turned to 180 degrees
- moved R4 62.4 mm to (106.8, 94.9), turned to 180 degrees
- moved R1 62.3 mm to (106.7, 72.0), turned to 180 degrees
- moved R2 62.3 mm to (106.7, 69.5), turned to 180 degrees
- moved R3 62.3 mm to (106.7, 74.5), turned to 180 degrees
- moved X1 52.5 mm to (107.1, 139.3)
- moved U2 52.5 mm to (102.0, 44.1)
- moved C2 42.7 mm to (122.7, 82.2), turned to 0 degrees
- moved C9 26.8 mm to (83.7, 45.1), turned to 180 degrees
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Routing:
- net D3: track 333.9 -> 0.00 mm, vias 3 -> 0
- net A1: track 323.5 -> 0.00 mm, vias 6 -> 0
- net D5: track 323.1 -> 0.00 mm, vias 4 -> 0
- net A2: track 316.2 -> 0.00 mm, vias 6 -> 0
- net D2: track 314.4 -> 0.00 mm, vias 2 -> 0
- net D4: track 313.7 -> 0.00 mm, vias 2 -> 0
- net A3: track 313.7 -> 0.00 mm, vias 4 -> 0
- net D1: track 312.6 -> 0.00 mm
- net D0: track 299.6 -> 0.00 mm, vias 1 -> 0
- net D7: track 299.1 -> 0.00 mm, vias 3 -> 0
- net D6: track 292.9 -> 0.00 mm, vias 6 -> 0
- net A4: track 267.4 -> 0.00 mm, vias 4 -> 0
- net R~{W}: track 256.4 -> 0.00 mm, vias 3 -> 0
- net D8: track 245.2 -> 0.00 mm, vias 2 -> 0
- net ~{RESET}: track 242.7 -> 0.00 mm, vias 3 -> 0
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- removed copper zone on B.Cu, net GND

Commit message: first plot
Parts:
- moved C11 77.4 mm to (118.6, 96.6)
- moved U10 77.4 mm to (108.2, 96.5)
- moved C1 57.6 mm to (49.3, 80.8), turned to 90 degrees
- moved C2 56.0 mm to (66.7, 84.1)
- moved R1 56.0 mm to (50.7, 73.9)
- moved R2 56.0 mm to (50.7, 71.4)
- moved R3 56.0 mm to (50.7, 76.5)
- moved R4 56.0 mm to (50.8, 96.8)
- moved R5 56.0 mm to (50.8, 99.2)
- moved X1 56.0 mm to (51.1, 141.2)
- moved U2 56.0 mm to (46.0, 46.0)
- moved U8 45.7 mm to (83.3, 46.0)
- moved C8 45.7 mm to (93.7, 46.1)
- moved C10 37.7 mm to (93.5, 96.5)
- moved U11 37.7 mm to (83.1, 96.5)
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Routing:
- net +5V: track 682.6 -> 133.5 mm, vias 1 -> 17
- net D4: track 0.00 -> 358.6 mm, vias 0 -> 1
- net D7: track 0.00 -> 319.6 mm, vias 0 -> 1
- net A1: track 0.00 -> 317.5 mm, vias 0 -> 4
- net D3: track 0.00 -> 311.7 mm, vias 0 -> 2
- net D2: track 0.00 -> 309.0 mm, vias 0 -> 2
- net A3: track 0.00 -> 303.0 mm, vias 0 -> 2
- net A2: track 0.00 -> 293.8 mm, vias 0 -> 2
- net D1: track 0.00 -> 291.8 mm, vias 0 -> 2
- net D0: track 0.00 -> 290.7 mm, vias 0 -> 1
- net ~{RESET}: track 0.00 -> 281.2 mm, vias 0 -> 1
- net D5: track 0.00 -> 272.0 mm, vias 0 -> 1
- net D6: track 0.00 -> 271.7 mm, vias 0 -> 2
- net D15: track 0.00 -> 266.2 mm
- net D13: track 0.00 -> 265.9 mm, vias 0 -> 1
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- added copper zone on In2.Cu, net +5V
- added copper zone on In1.Cu, net GND
Other:
- copper layers 2 -> 4
- board text removed: "CONSOLE"
