File: rev1/schematic/raven68k-rev1/raven68k-rev1.kicad_pcb (KiCad board)
At the start: 4 copper layers, 203.2 x 114.3 mm, 78 parts, among them IC1 L5970D013TR, IC2 L5970D013TR, J1 CPLD_JTAG, J2 DUART_IO, J3 RAPC722BK, SW1 RESET_SW, U1 MCP100-465D, U10 28C256, U11 28C256, U2 68010D, U3 XC9572XL-VQ44, U4 68681, U5 74LS373, U6 CONSOLE, U7 DS12887+, U8 KM684000BLP-7L, U9 KM684000BLP-7L, X1 CLOCK, X2 CXO_DIP14

Commit message: add board standoffs
Parts:
- added REF**: MountingHole_4mm, MountingHole:MountingHole_4mm, F.Cu at (40.6, 146.8)
- added REF**: MountingHole_4mm, MountingHole:MountingHole_4mm, F.Cu at (238.8, 146.6)
- added REF**: MountingHole_4mm, MountingHole:MountingHole_4mm, F.Cu at (237.7, 72.1)
- added REF**: MountingHole_4mm, MountingHole:MountingHole_4mm, F.Cu at (40.1, 42.7)
Other:
- board size 203.2 x 114.3 mm -> 208.3 x 114.3 mm
- board text added: "JLCPCB Order No."
- board text removed: "Order No."
Changed lines of the file:
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@@
     )
   )
+  (footprint "MountingHole:MountingHole_4mm" (layer "F.Cu")
+    (at 40.64 146.812)
+    (descr "Mounting Hole 4mm, no annular")
+    (tags "mounting hole 4mm no annular")
+    (attr exclude_from_pos_files exclude_from_bom)
+    (fp_text reference "REF**" (at 0 -5) (layer "F.SilkS")
+      (effects (font (size 1 1) (thickness 0.15)))
+    )
+    (fp_text value "MountingHole_4mm" (at 0 5) (layer "F.Fab")
+      (effects (font (size 1 1) (thickness 0.15)))
+    )
+    (fp_text user "${REFERENCE}" (at 0.3 0) (layer "F.Fab")
+      (effects (font (size 1 1) (thickness 0.15)))
+    )
+    (fp_circle (center 0 0) (end 4 0) (layer "Cmts.User") (width 0.15) (fill none))
+    (fp_circle (center 0 0) (end 4.25 0) (layer "F.CrtYd") (width 0.05) (fill none))
+    (pad "" np_thru_hole circle (at 0 0) (size 4 4) (drill 4) (layers *.Cu *.Mask))
+  )
   (footprint "Package_SO:SO-8_5.3x6.2mm_P1.27mm" (layer "F.Cu")
     (at 198.12 54.61)
@@
     )
   )
+  (footprint "MountingHole:MountingHole_4mm" (layer "F.Cu")
+    (at 238.76 146.558)
+    (descr "Mounting Hole 4mm, no annular")
+    (tags "mounting hole 4mm no annular")
+    (attr exclude_from_pos_files exclude_from_bom)
+    (fp_text reference "REF**" (at 0 -5) (layer "F.SilkS")
+      (effects (font (size 1 1) (thickness 0.15)))
+    )
+    (fp_text value "MountingHole_4mm" (at 0 5) (layer "F.Fab")
+      (effects (font (size 1 1) (thickness 0.15)))
+    )
+    (fp_text user "${REFERENCE}" (at 0.3 0) (layer "F.Fab")
+      (effects (font (size 1 1) (thickness 0.15)))
+    )
+    (fp_circle (center 0 0) (end 4 0) (layer "Cmts.User") (width 0.15) (fill none))
+    (fp_circle (center 0 0) (end 4.25 0) (layer "F.CrtYd") (width 0.05) (fill none))
+    (pad "" np_thru_hole circle (at 0 0) (size 4 4) (drill 4) (layers *.Cu *.Mask))
+  )
   (footprint "raven68k-rev1:GPTS203212B" (layer "F.Cu")
     (at 232.283 45.974 180)
@@
     )
   )
+  (footprint "MountingHole:MountingHole_4mm" (layer "F.Cu")
+    (at 237.744 72.136)
+    (descr "Mounting Hole 4mm, no annular")
+    (tags "mounting hole 4mm no annular")
+    (attr exclude_from_pos_files exclude_from_bom)
+    (fp_text reference "REF**" (at 0 -5) (layer "F.SilkS")
+      (effects (font (size 1 1) (thickness 0.15)))
+    )
+    (fp_text value "MountingHole_4mm" (at 0 5) (layer "F.Fab")
+      (effects (font (size 1 1) (thickness 0.15)))
+    )
+    (fp_text user "${REFERENCE}" (at 0.3 0) (layer "F.Fab")
+      (effects (font (size 1 1) (thickness 0.15)))
+    )
+    (fp_circle (center 0 0) (end 4 0) (layer "Cmts.User") (width 0.15) (fill none))
+    (fp_circle (center 0 0) (end 4.25 0) (layer "F.CrtYd") (width 0.05) (fill none))
+    (pad "" np_thru_hole circle (at 0 0) (size 4 4) (drill 4) (layers *.Cu *.Mask))
+  )
+  (footprint "MountingHole:MountingHole_4mm" (layer "F.Cu")
+    (at 40.132 42.672)
+    (descr "Mounting Hole 4mm, no annular")
+    (tags "mounting hole 4mm no annular")
+    (attr exclude_from_pos_files exclude_from_bom)
+    (fp_text reference "REF**" (at 5.842 -3.048) (layer "F.SilkS")
+      (effects (font (size 1 1) (thickness 0.15)))
+    )
+    (fp_text value "MountingHole_4mm" (at 0 5) (layer "F.Fab")
+      (effects (font (size 1 1) (thickness 0.15)))
+    )
+    (fp_text user "${REFERENCE}" (at 0.3 0) (layer "F.Fab")
+      (effects (font (size 1 1) (thickness 0.15)))
+    )
+    (fp_circle (center 0 0) (end 4 0) (layer "Cmts.User") (width 0.15) (fill none))
+    (fp_circle (center 0 0) (end 4.25 0) (layer "F.CrtYd") (width 0.05) (fill none))
+    (pad "" np_thru_hole circle (at 0 0) (size 4 4) (drill 4) (layers *.Cu *.Mask))
+  )
   (footprint "Resistor_SMD:R_1206_3216Metric_Pad1.30x1.75mm_HandSolder" (layer "F.Cu")
     (at 189.23 60.96 -90)
@@
     (fp_line (start -1.6 -0.8) (end 1.6 -0.8) (layer "F.Fab") (width 0.1))
     (fp_line (start -1.6 0.8) (end -1.6 -0.8) (layer "F.Fab") (width 0.1))
-    (pad "1" smd roundrect (at -1.5625 0) (size 1.325 1.8) (layers "F.Cu" "F.Paste" "F.Mask") (roundrect_rratio 0.188679)
+    (pad "1" smd roundrect (at -1.5625 0) (size 1.325 1.8) (layers "F.Cu" "F.Paste" "F.Mask") (roundrect_rratio 0.1886792453)
       (net 22 "GND") (pintype "passive"))
-    (pad "2" smd roundrect (at 1.5625 0) (size 1.325 1.8) (layers "F.Cu" "F.Paste" "F.Mask") (roundrect_rratio 0.188679)
+    (pad "2" smd roundrect (at 1.5625 0) (size 1.325 1.8) (layers "F.Cu" "F.Paste" "F.Mask") (roundrect_rratio 0.1886792453)
       (net 25 "+5V") (pintype "passive"))
     (model "${KICAD6_3DMODEL_DIR}/Capacitor_SMD.3dshapes/C_1206_3216Metric.wrl"
@@
     )
   )
-  (gr_line (start 38.1 152.4) (end 38.1 38.1) (layer "Edge.Cuts") (width 0.05))
-  (gr_line (start 241.3 38.1) (end 241.3 152.4) (layer "Edge.Cuts") (width 0.05))
-  (gr_line (start 241.3 152.4) (end 38.1 152.4) (layer "Edge.Cuts") (width 0.05))
-  (gr_line (start 38.1 38.1) (end 241.3 38.1) (layer "Edge.Cuts") (width 0.05))
-  (gr_text "Order No. " (at 66.04 149.86) (layer "B.SilkS")
+  (gr_line (start 35.56 152.4) (end 35.56 38.1) (layer "Edge.Cuts") (width 0.05))
+  (gr_line (start 243.84 38.1) (end 243.84 152.4) (layer "Edge.Cuts") (width 0.05))
+  (gr_line (start 243.84 152.4) (end 35.56 152.4) (layer "Edge.Cuts") (width 0.05))
+  (gr_line (start 35.56 38.1) (end 243.84 38.1) (layer "Edge.Cuts") (width 0.05))
+  (gr_text "JLCPCB Order No. " (at 70.612 149.86) (layer "B.SilkS")
     (effects (font (size 1.5 1.5) (thickness 0.3)) (justify mirror))
   )
@@
     (effects (font (size 1 1) (thickness 0.15)))
   )
-  (gr_text "The Raven68k (Rev 1, 2022-02-09) https://github.com/jkuituni/Raven68k" (at 209.042 149.606) (layer "F.SilkS")
+  (gr_text "The Raven68k (Rev 1, 2022-02-09) https://github.com/jkuituni/Raven68k" (at 198.374 149.606) (layer "F.SilkS")
     (effects (font (size 1 1) (thickness 0.15)))
   )
@@
     (connect_pads (clearance 0.508))
     (min_thickness 0.254) (filled_areas_thickness no)
-    (fill yes (thermal_gap 0.508) (thermal_bridge_width 0.508))
+    (fill (thermal_gap 0.508) (thermal_bridge_width 0.508))
     (polygon
       (pts
-        (xy 241.3 152.4)
+        (xy 244.094 152.4)
         (xy 38.1 152.4)
-        (xy 37.846 152.146)
-        (xy 38.1 38.1)
-        (xy 241.3 38.1)
+        (xy 35.052014 152.139778)
+        (xy 35.306014 38.093778)
+        (xy 244.094 38.1)
       )
     )
@@
     (polygon
       (pts
-        (xy 241.808 38.354)
-        (xy 241.046 152.654)
-        (xy 38.1 152.654)
-        (xy 38.1 38.1)
+        (xy 244.347887 38.370933)
+        (xy 243.585887 152.670933)
+        (xy 35.052 152.654)
+        (xy 35.052 38.1)
       )
     )
