File: rev1/schematic/raven68k-rev1/DUART.kicad_sch (KiCad schematic)
At the start: 12 parts, among them J2 DUART_IO, U4 68681, U5 74LS373, U6 CONSOLE, U7 DS12887+, X2 CXO_DIP14

Commit message: some helpful labels
Parts:
- C5, C6, C7: LCSC (none) -> C24497
Changed lines of the file:
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@@
+      (effects (font (size 1.27 1.27)) hide)
+    )
+    (property "LCSC" "C24497" (id 4) (at 68.58 163.83 0)
       (effects (font (size 1.27 1.27)) hide)
     )
@@
       (effects (font (size 1.27 1.27)) hide)
     )
+    (property "LCSC" "C24497" (id 4) (at 80.01 163.83 0)
+      (effects (font (size 1.27 1.27)) hide)
+    )
     (pin "1")
     (pin "2")
@@
       (effects (font (size 1.27 1.27)) hide)
     )
+    (property "LCSC" "C24497" (id 4) (at 91.44 163.83 0)
+      (effects (font (size 1.27 1.27)) hide)
+    )

Commit message: naming update for NOT_LDS
Connections:
- net NOT_DS renamed NOT_LDS
Changed lines of the file:
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@@
     (effects (font (size 1.27 1.27)) (justify right))
   )
-  (hierarchical_label "NOT_DS" (shape input) (at 247.65 118.11 0)
+  (hierarchical_label "NOT_LDS" (shape input) (at 247.65 118.11 0)
     (effects (font (size 1.27 1.27)) (justify left))
   )
