File: rev1/schematic/raven68k-rev1/raven68k-rev1.kicad_sch (KiCad schematic)
At the start: 15 parts, among them J1 CPLD_JTAG, SW1 RESET_SW, U1 MCP100-465D, U2 68010D, U3 XC9572XL-VQ44, X1 CLOCK

Commit message: board layout complete, needs verification
Parts:
- removed SW1: RESET_SW, raven68k-rev1:TS0266170BK160SCRD, symbol Switch:SW_Push
- added S1: RESET_SW, raven68k-rev1:TS0266170BK160SCRD, symbol custom:TS02-66-170-BK-160-SCR-D
Connections:
- net +5V: now also S1.1 (NO_1), S1.2 (NO_2)
- net GND: now also S1.3 (COM_1), S1.4 (COM_2)

Commit message: move components around
Parts:
- removed S1: RESET_SW, raven68k-rev1:TS0266170BK160SCRD, symbol custom:TS02-66-170-BK-160-SCR-D
- added SW1: RESET_SW, raven68k-rev1:TS0266170BK160SCRD, symbol custom:TS02-66-170-BK-160-SCR-D
Connections:
- net +5V: now also SW1.1 (NO_1), SW1.2 (NO_2)
- net GND: now also SW1.3 (COM_1), SW1.4 (COM_2)

Commit message: some helpful labels
Parts:
- added C28: 0.1uF, Capacitor_SMD:C_1206_3216Metric_Pad1.33x1.80mm_HandSolder, symbol Device:C_Small
- C1, C2, C3, C4: LCSC (none) -> C24497
Connections:
- net +5V: now also C28.2
- net GND: now also C28.1
Changed lines of the file:
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@@
   (junction (at 43.18 80.01) (diameter 0) (color 0 0 0 0)
+  )
+  (junction (at 171.45 154.94) (diameter 0) (color 0 0 0 0)
+  )
+  (junction (at 171.45 149.86) (diameter 0) (color 0 0 0 0)
   )
   (junction (at 201.93 149.86) (diameter 0) (color 0 0 0 0)
@@
     (stroke (width 0) (type default) (color 0 0 0 0))
   )
+  (wire (pts (xy 171.45 149.86) (xy 180.34 149.86))
+    (stroke (width 0) (type default) (color 0 0 0 0))
+  )
   (wire (pts (xy 45.72 85.09) (xy 45.72 82.55))
     (stroke (width 0) (type default) (color 0 0 0 0))
@@
   )
   (wire (pts (xy 119.38 100.33) (xy 115.57 100.33))
+    (stroke (width 0) (type default) (color 0 0 0 0))
+  )
+  (wire (pts (xy 171.45 154.94) (xy 180.34 154.94))
     (stroke (width 0) (type default) (color 0 0 0 0))
   )
@@
       (effects (font (size 1.27 1.27)) hide)
     )
+    (property "LCSC" "C24497" (id 4) (at 162.56 152.4 90)
+      (effects (font (size 1.27 1.27)) hide)
+    )
     (pin "1")
     (pin "2")
@@
       (effects (font (size 1.27 1.27)) hide)
     )
+    (property "LCSC" "C24497" (id 4) (at 171.45 152.4 90)
+      (effects (font (size 1.27 1.27)) hide)
+    )
     (pin "1")
     (pin "2")
@@
       (effects (font (size 1.27 1.27)) hide)
     )
+    (property "LCSC" "C24497" (id 4) (at 201.93 152.4 90)
+      (effects (font (size 1.27 1.27)) hide)
+    )
     (pin "1")
     (pin "2")
@@
     )
     (property "Datasheet" "~" (id 3) (at 210.82 152.4 0)
+      (effects (font (size 1.27 1.27)) hide)
+    )
+    (property "LCSC" "C24497" (id 4) (at 210.82 152.4 90)
       (effects (font (size 1.27 1.27)) hide)
     )
@@
     (pin "1")
   )
+  (symbol (lib_id "Device:C_Small") (at 180.34 152.4 180) (unit 1)
+    (in_bom yes) (on_board yes)
+    (property "Reference" "C28" (id 0) (at 186.1566 152.4 90))
+    (property "Value" "0.1uF" (id 1) (at 183.8452 152.4 90))
+    (property "Footprint" "Capacitor_SMD:C_1206_3216Metric_Pad1.33x1.80mm_HandSolder" (id 2) (at 180.34 152.4 0)
+      (effects (font (size 1.27 1.27)) hide)
+    )
+    (property "Datasheet" "~" (id 3) (at 180.34 152.4 0)
+      (effects (font (size 1.27 1.27)) hide)
+    )
+    (property "LCSC" "C24497" (id 4) (at 180.34 152.4 90)
+      (effects (font (size 1.27 1.27)) hide)
+    )
+    (pin "1")
+    (pin "2")
+  )
   (sheet (at 27.94 16.51) (size 24.13 20.32) (fields_autoplaced)
     (stroke (width 0) (type solid) (color 0 0 0 0))
@@
     )
     (path "/00000000-0000-0000-0000-00006263c73f/00000000-0000-0000-0000-00006268364e"
-      (reference "C26") (unit 1) (value "100nF") (footprint "Capacitor_SMD:C_1206_3216Metric_Pad1.33x1.80mm_HandSolder")
+      (reference "C26") (unit 1) (value "0.1uF") (footprint "Capacitor_SMD:C_1206_3216Metric_Pad1.33x1.80mm_HandSolder")
     )
     (path "/00000000-0000-0000-0000-00006263c73f/00000000-0000-0000-0000-0000626b0fd3"
-      (reference "C27") (unit 1) (value "100nF") (footprint "Capacitor_SMD:C_1206_3216Metric_Pad1.33x1.80mm_HandSolder")
+      (reference "C27") (unit 1) (value "0.1uF") (footprint "Capacitor_SMD:C_1206_3216Metric_Pad1.33x1.80mm_HandSolder")
+    )
+    (path "/f89b44fd-1fe0-4315-acaa-6aedbac4e8d4"
+      (reference "C28") (unit 1) (value "0.1uF") (footprint "Capacitor_SMD:C_1206_3216Metric_Pad1.33x1.80mm_HandSolder")
     )
     (path "/00000000-0000-0000-0000-00006263c73f/00000000-0000-0000-0000-00006263e7cb"

Commit message: naming update for NOT_LDS
Connections:
- net NOT_DS renamed NOT_LDS
Other:
- sheet DUART and RTC ports: added NOT_LDS; removed NOT_DS
Changed lines of the file:
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@@
     )
   )
-  (global_label "NOT_DS" (shape output) (at 160.02 102.87 180) (fields_autoplaced)
-    (effects (font (size 1.27 1.27)) (justify right))
-    (property "Intersheet References" "${INTERSHEET_REFS}" (id 0) (at 0 0 0)
-      (effects (font (size 1.27 1.27)) hide)
+  (global_label "NOT_LDS" (shape output) (at 160.02 102.87 180) (fields_autoplaced)
+    (effects (font (size 1.27 1.27)) (justify right))
+    (property "Intersheet References" "${INTERSHEET_REFS}" (id 0) (at 149.592 102.7906 0)
+      (effects (font (size 1.27 1.27)) (justify right) hide)
     )
   )
@@
     )
   )
-  (global_label "NOT_DS" (shape input) (at 83.82 41.91 180) (fields_autoplaced)
-    (effects (font (size 1.27 1.27)) (justify right))
-    (property "Intersheet References" "${INTERSHEET_REFS}" (id 0) (at 0 0 0)
-      (effects (font (size 1.27 1.27)) hide)
+  (global_label "NOT_LDS" (shape input) (at 83.82 41.91 180) (fields_autoplaced)
+    (effects (font (size 1.27 1.27)) (justify right))
+    (property "Intersheet References" "${INTERSHEET_REFS}" (id 0) (at 73.392 41.8306 0)
+      (effects (font (size 1.27 1.27)) (justify right) hide)
     )
   )
@@
       (effects (font (size 1.27 1.27)) (justify left))
     )
-    (pin "NOT_DS" input (at 87.63 41.91 180)
-      (effects (font (size 1.27 1.27)) (justify left))
-    )
     (pin "~{IPL1}" output (at 111.76 34.29 0)
       (effects (font (size 1.27 1.27)) (justify right))
@@
       (effects (font (size 1.27 1.27)) (justify left))
     )
+    (pin "NOT_LDS" input (at 87.63 41.91 180)
+      (effects (font (size 1.27 1.27)) (justify left))
+    )
